File: msxbuspcb/_autosave-msxbus.kicad_pcb (KiCad board)
At the start: 2 copper layers, 9 parts, among them J1 RPi_GPIO, P1 CONN_02X25, P2 CONN_02X25, P4 CONN_01X03, U1 EMP240

Commit message: update for RPMC
Parts:
- added P3: CONN_02X05, Pin_Headers:Pin_Header_Straight_2x05, F.Cu at (175.2, 92.8)
- R1, R2, R3, R4: footprint Resistors_SMD:R_2010_HandSoldering -> Resistors_SMD:R_0603_HandSoldering
- moved R1 16.7 mm to (176.5, 89.6)
- moved R2 4.48 mm to (180.9, 93.3), turned to 270 degrees
- moved R3 3.66 mm to (180.9, 98.0), turned to 90 degrees
- moved R4 2.93 mm to (181.0, 102.8), turned to 270 degrees
