File: msxslot/msxslotpi.kicad_pcb (KiCad board)
At the start: 2 copper layers, 7 parts, among them J1 RPi_GPIO, P1 CONN_02X25, U1 74LS595, U2 74LS595, U3 74LS595, U4 74LS165, U5 74LS165

Commit message: add feature with Altera CPLD EMP240
Parts:
- added P2: SLOT 2, Pin_Headers:Pin_Header_Straight_2x25, F.Cu at (166.4, 125.7)
- added P3: UART, Pin_Headers:Pin_Header_Angled_1x04, F.Cu at (170.2, 91.4)
- P1: value CONN_02X25 -> SLOT 1
- moved P1 24.4 mm to (166.4, 143.5)
Connections:
- net Net-(J1-Pad38) renamed /STLSL2
- J1 pad 1: /3V3 -> VCC
- J1 pad 10: Net-(J1-Pad10) -> /RXD
- J1 pad 13: Net-(J1-Pad13) -> /SLOTSW
- J1 pad 17: /3V3 -> VCC
- J1 pad 29: Net-(J1-Pad29) -> /SLOT1
- J1 pad 31: Net-(J1-Pad31) -> /SLOT2
- J1 pad 8: Net-(J1-Pad8) -> /TXD
- P1 pad 44: Net-(P1-Pad44) -> /SLOT1
- P1 pad 46: Net-(P1-Pad46) -> /SLOTSW
- U1 pad 10: /3V3 -> VCC
- U2 pad 10: /3V3 -> VCC
- U3 pad 10: /3V3 -> VCC
Routing:
- net /5V: track 0.00 -> 181.4 mm
- net /CS12: track 0.00 -> 169.0 mm
- net /CLK: track 0.00 -> 149.1 mm, vias 0 -> 2
- net /WR: track 0.00 -> 147.2 mm, vias 0 -> 2
- net /SLOTSW: track 0.00 -> 142.4 mm
- net /SLTSL: track 0.00 -> 129.1 mm, vias 0 -> 4
- net VCC: track 0.00 -> 125.0 mm
- net /SLOT1: track 0.00 -> 117.7 mm, vias 0 -> 1
- net /CS1: track 0.00 -> 111.6 mm, vias 0 -> 1
- net /SLOT2: track 0.00 -> 97.4 mm, vias 0 -> 1
- net /RD: track 0.00 -> 96.2 mm
- net /D1: track 0.00 -> 76.9 mm, vias 0 -> 2
- net /D2: track 0.00 -> 65.9 mm, vias 0 -> 7
- net /D6: track 0.00 -> 60.6 mm, vias 0 -> 3
- net /A08: track 0.00 -> 58.1 mm, vias 0 -> 2
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- added copper zone on B.Cu, net GND
- added copper zone on F.Cu, net GND
