File: rpspc/rpspc.sch (KiCad schematic (older format))
At the start: 4 parts, among them J1 RPi_GPIO, J2 Conn_02x17_Top_Bottom, U1 74LS245, U2 74LS245

Commit message: modification for rpmcv4 and rpibox
Parts:
- J2: footprint rpspc:cardedge_female_2x17_2.54mm -> Socket_Strips:Socket_Strip_Straight_2x20_Pitch2.54mm
Connections:
- wire segments 106 -> 105
Changed lines of the file:
@@
 F 0 "J2" H 2500 4100 50  0000 C CNN
 F 1 "Conn_02x17_Top_Bottom" H 2500 2300 50  0000 C CNN
-F 2 "rpspc:cardedge_female_2x17_2.54mm" H 2450 3200 50  0001 C CNN
+F 2 "Socket_Strips:Socket_Strip_Straight_2x20_Pitch2.54mm" H 2450 3200 50  0001 C CNN
 F 3 "" H 2450 3200 50  0001 C CNN
 	1    2450 3200
@@
 	3100 3600 2750 3600
 Wire Wire Line
-	3100 4000 2750 4000
+	2750 4000 3570 4000
 Wire Wire Line
 	4390 1835 4840 1835
@@
 	10300 2600 10750 2600
 Wire Wire Line
-	10850 2200 10300 2200
-Wire Wire Line
-	10300 2100 10850 2100
-Wire Wire Line
 	10300 2300 10850 2300
 Wire Wire Line
@@
 	10300 3000 10750 3000
 Wire Wire Line
-	10300 3700 10850 3700
+	10850 3700 10300 3700
 Wire Wire Line
 	7800 4000 8400 4000
@@
 L GND #PWR03
 U 1 1 5A410041
-P 11150 4350
-F 0 "#PWR03" H 11150 4100 50  0001 C CNN
-F 1 "GND" H 11150 4200 50  0000 C CNN
-F 2 "" H 11150 4350 50  0001 C CNN
-F 3 "" H 11150 4350 50  0001 C CNN
-	1    11150 4350
+P 10850 4145
+F 0 "#PWR03" H 10850 3895 50  0001 C CNN
+F 1 "GND" H 10850 3995 50  0000 C CNN
+F 2 "" H 10850 4145 50  0001 C CNN
+F 3 "" H 10850 4145 50  0001 C CNN
+	1    10850 4145
 	1    0    0    -1
 $EndComp
-Wire Wire Line
-	11150 2500 11150 4350
-Connection ~ 11150 3900
-Connection ~ 11150 3700
-Connection ~ 11150 2900
 Wire Wire Line
 	7800 2500 7800 4000
@@
 Connection ~ 7800 3300
 Wire Wire Line
-	10300 3500 10850 3500
+	10850 3500 10300 3500
 Wire Wire Line
 	8400 3300 7800 3300
@@
 L +5V #PWR04
 U 1 1 5A4104BD
-P 11150 1900
-F 0 "#PWR04" H 11150 1750 50  0001 C CNN
-F 1 "+5V" H 11150 2040 50  0000 C CNN
-F 2 "" H 11150 1900 50  0001 C CNN
-F 3 "" H 11150 1900 50  0001 C CNN
-	1    11150 1900
+P 10850 1940
+F 0 "#PWR04" H 10850 1790 50  0001 C CNN
+F 1 "+5V" H 10850 2080 50  0000 C CNN
+F 2 "" H 10850 1940 50  0001 C CNN
+F 3 "" H 10850 1940 50  0001 C CNN
+	1    10850 1940
 	1    0    0    -1
 $EndComp
-Wire Wire Line
-	11150 1900 11150 2400
-Connection ~ 11150 2300
 Wire Wire Line
 	8400 2700 7950 2700
@@
 	6690 1260 6690 1635
 Wire Wire Line
-	3100 4005 3570 4005
-Wire Wire Line
-	3570 4005 3570 1260
+	3570 1260 3570 4110
 Wire Wire Line
 	3570 1260 6690 1260
 Connection ~ 6690 1535
+Wire Wire Line
+	10850 2300 10850 4145
+Connection ~ 10850 3500
+Connection ~ 10850 2700
+Connection ~ 3570 4000
+$Comp
+L GND #PWR05
+U 1 1 5A5CCD83
+P 3570 4110
+F 0 "#PWR05" H 3570 3860 50  0001 C CNN
+F 1 "GND" H 3570 3960 50  0000 C CNN
+F 2 "" H 3570 4110 50  0001 C CNN
+F 3 "" H 3570 4110 50  0001 C CNN
+	1    3570 4110
+	1    0    0    -1
+$EndComp
+Wire Wire Line
+	10850 1940 10850 2200
+Connection ~ 10850 2200
+Wire Wire Line
+	10850 2200 10300 2200
+Wire Wire Line
+	10300 2100 10850 2100
+Connection ~ 10850 2100
+Connection ~ 10850 3700
 $EndSCHEMATC
