File: mos6502/6502.kicad_pcb (KiCad board)
At the start: 2 copper layers, 4 parts, among them U2 74HC245, U3 74HC245, U4 74HC245, U5 WD65C02

Commit message: update for PCB order
Parts:
- added C1: C, Capacitors_SMD:C_0603_HandSoldering, F.Cu at (146.1, 95.2)
- added C2: C, Capacitors_SMD:C_0603_HandSoldering, F.Cu at (188.0, 95.2)
- added C3: C, Capacitors_SMD:C_0603_HandSoldering, B.Cu at (146.1, 95.2)
- added C4: C, Capacitors_SMD:C_0603_HandSoldering, B.Cu at (188.0, 95.2)
- added C5: C, Capacitors_SMD:C_0603_HandSoldering, B.Cu at (158.8, 77.5)
- added D1: LED, Capacitors_SMD:C_0603_HandSoldering, F.Cu at (138.4, 104.1)
- added D2: LED, Capacitors_SMD:C_0603_HandSoldering, F.Cu at (194.3, 104.1)
- added J1: Raspberry_Pi_2_3, Pin_Headers:Pin_Header_Straight_2x20, F.Cu at (190.8, 113.3)
- added R1: R, Capacitors_SMD:C_0603_HandSoldering, B.Cu at (194.3, 104.1)
- added R2: R, Capacitors_SMD:C_0603_HandSoldering, B.Cu at (138.4, 104.1)
- added REF**: RPi_Hat_PTH, msx:z_RPi_Hat_layout, F.Cu at (166.7, 90.1)
- added U1: 74HC245, Housings_SOIC:SOIC-20W_7.5x12.8mm_Pitch1.27mm, B.Cu at (178.2, 95.6)
- U3: moved to B.Cu
- U5: footprint Housings_DIP:DIP-40_W25.4mm_LongPads -> Housings_DIP:DIP-40_W15.24mm_LongPads
- moved U5 49.7 mm to (142.6, 80.5), turned to 90 degrees
- moved U4 41.8 mm to (178.2, 95.6), turned to 90 degrees
- moved U2 36.4 mm to (155.4, 95.6), turned to 90 degrees
- moved U3 19.5 mm to (155.4, 95.6), turned to 270 degrees
Connections:
- U2 pad 1: GND -> VCC
- U5 pad 4: /NC -> /IRQ
Routing:
- net GND: track 0.00 -> 256.5 mm, vias 0 -> 2
- net VCC: track 0.00 -> 137.7 mm, vias 0 -> 2
- net /3V3: track 0.00 -> 88.0 mm, vias 0 -> 2
- net Net-(D2-Pad2): track 0.00 -> 79.8 mm, vias 0 -> 1
- net Net-(D1-Pad2): track 0.00 -> 79.2 mm, vias 0 -> 1
- net /RC24: track 0.00 -> 68.7 mm, vias 0 -> 1
- net /RD0: track 0.00 -> 50.9 mm
- net /RD6: track 0.00 -> 50.7 mm, vias 0 -> 1
- net /RC18: track 0.00 -> 50.1 mm, vias 0 -> 1
- net /RD2: track 0.00 -> 48.4 mm, vias 0 -> 1
- net /RD3: track 0.00 -> 45.7 mm, vias 0 -> 1
- net /RW: track 0.00 -> 45.1 mm, vias 0 -> 1
- net /RD7: track 0.00 -> 42.8 mm, vias 0 -> 1
- net /RD5: track 0.00 -> 41.7 mm, vias 0 -> 1
- net /RD4: track 0.00 -> 40.9 mm, vias 0 -> 2
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- added copper zone on B.Cu, net GND
- added copper zone on F.Cu, net GND
Other:
- board outline added: 65 x 56.5 mm
- net class VCC added: clearance 0.2, trace_width 0.35, via_dia 0.6, via_drill 0.4
- board text added: "2018.03.27"
- board text added: "74HC245"
- board text added: "MOS 6502"
- board text added: "READ"
- board text added: "Real 6502 Processor Engine V1.0 [6502BOX]"
- board text added: "WRITE"
- board text added: "meeso.kim@gmail.com 2018.03.27"

Commit message: minor update for PCB order
Parts:
- U1: value 74HC245 -> 74HC244; moved to F.Cu
- U2, U4: value 74HC245 -> 74HC244
- moved C2 12.8 mm to (175.3, 96.5)
- moved C4 12.8 mm to (175.3, 96.5)
- moved U4 11.9 mm to (166.4, 96.5), turned to 270 degrees
- moved C1 11.5 mm to (157.5, 96.5)
- moved C3 11.5 mm to (157.5, 96.5)
- moved U3 11.0 mm to (166.4, 96.5)
- moved U2 6.85 mm to (148.6, 96.5), turned to 270 degrees
- moved U1 5.97 mm to (184.2, 96.5), turned to 270 degrees
Connections:
- U1 pad 1: GND -> /RC24
- U1 pad 10: GND -> Net-(U1-Pad10)
- U1 pad 12: /A14 -> /RA11
- U1 pad 13: /A13 -> /A14
- U1 pad 14: /A12 -> /RA10
- U1 pad 15: /A11 -> /A13
- U1 pad 16: /A10 -> /RA9
- U1 pad 17: /A9 -> /A12
- U1 pad 18: /A8 -> /RA8
- U1 pad 2: /RA8 -> /A8
- U1 pad 20: VCC -> Net-(U1-Pad20)
- U1 pad 3: /RA9 -> /RA12
- U1 pad 4: /RA10 -> /A9
- U1 pad 5: /RA11 -> /RA13
- U1 pad 6: /RA12 -> /A10
- U1 pad 7: /RA13 -> /RA14
- U1 pad 8: /RA14 -> /A11
- U2 pad 1: VCC -> GND
- U2 pad 10: GND -> Net-(U2-Pad10)
- U2 pad 11: /RC23 -> /RW
- U2 pad 12: /IRQ -> /RESET
- U2 pad 13: /NMI -> /RC19
- U2 pad 14: /RC22 -> /RC21
- U2 pad 15: /RESET -> /RC18
- U2 pad 16: /RC21 -> /PHI0
- U2 pad 17: /PHI0 -> /SYNC
- U2 pad 20: VCC -> Net-(U2-Pad20)
- U2 pad 3: /RC20 -> /RC22
- U2 pad 4: /PHI2o -> /RC20
- U2 pad 5: /RC17 -> /NMI
- U2 pad 6: /SYNC -> /PHI2o
- U2 pad 7: /RC18 -> /IRQ
- U2 pad 8: /RC19 -> /RC17
- U2 pad 9: /RW -> /RC23
- U4 pad 1: GND -> /RC24
- U4 pad 10: GND -> Net-(U4-Pad10)
- U4 pad 12: /A6 -> /RD3
- U4 pad 13: /A5 -> /A6
- U4 pad 14: /A4 -> /RD2
- U4 pad 15: /A3 -> /A5
- U4 pad 16: /A2 -> /RD1
- U4 pad 17: /A1 -> /A4
- U4 pad 18: /A0 -> /RD0
- U4 pad 2: /RD0 -> /A0
- U4 pad 20: VCC -> Net-(U4-Pad20)
- U4 pad 3: /RD1 -> /RD4
- U4 pad 4: /RD2 -> /A1
- U4 pad 5: /RD3 -> /RD5
- U4 pad 6: /RD4 -> /A2
- U4 pad 7: /RD5 -> /RD6
- U4 pad 8: /RD6 -> /A3
Routing:
- net VCC: track 137.7 -> 74.7 mm
- net /RA13: track 33.7 -> 89.5 mm, vias 1 -> 0
- net Net-(D2-Pad2): track 79.8 -> 125.8 mm
- net /RW: track 45.1 -> 84.9 mm
- net /A7: track 11.8 -> 40.2 mm
- net /RA12: track 35.3 -> 62.9 mm
- net /PHI0: track 28.0 -> 49.5 mm
- net /SYNC: track 22.8 -> 42.8 mm
- net GND: track 256.5 -> 237.8 mm
- net /RDY: track 13.4 -> 31.7 mm
- net /RA14: track 27.8 -> 45.3 mm
- net /A6: track 12.3 -> 29.7 mm, vias 0 -> 1
- net /A5: track 12.8 -> 29.7 mm
- net /A8: track 11.9 -> 28.0 mm, vias 1 -> 0
- net /RD0: track 50.9 -> 35.7 mm
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Other:
- board text added: "74HC244"
