File: rpiapplev2/rpiapple.kicad_pcb (KiCad board)
At the start: 2 copper layers, 81.3 x 74.9 mm, 21 parts, among them J1 Raspberry_Pi_2_3, J2 Raspberry_Pi_2_3, P1 A2Bus, U1 LVC4245, U2 74LS05, U3 74HC244, U4 74HC244, U5 74HC244, U6 74LS08

Commit message: SPC/APPLE/RPMC/RPMP updated for PCB order
Parts:
- added G1: LOGO, MSX:raspberry_pi_logo, B.Cu at (119.4, 96.5)
- added G2: LOGO, MSX:appleii_logo, B.Cu at (145.4, 94.0)
- added G3: LOGO, MSX:appleii_logo, F.Cu at (165.1, 105.4)
- U1: footprint Housings_SOIC:SOIC-24W_7.5x15.4mm_Pitch1.27mm -> SMD_Packages:SOIC-24
- moved C7 65.0 mm to (137.2, 121.0), turned to 90 degrees
- moved G4 11.5 mm to (114.9, 104.1)
- moved C5 1.77 mm to (137.2, 115.9), turned to 270 degrees
- moved C4 0.30 mm to (137.2, 117.9), turned to 270 degrees
- turned U1 to 180 degrees
- renumbered G*** to G4
Connections:
- C1 pad 1: VCC -> /3V3
- C2 pad 1: VCC -> /3V3
- C3 pad 1: VCC -> /3V3
- C4 pad 1: VCC -> /3V3
- C5 pad 1: VCC -> /3V3
- C6 pad 1: VCC -> /3V3
- C7 pad 1: /3V3 -> VCC
- U1 pad 23: Net-(U1-Pad23) -> /3V3
Routing:
- net GND: track 0.00 -> 296.3 mm, vias 0 -> 4
- net /3V3: track 0.00 -> 203.1 mm, vias 0 -> 4
- net /DAT_DIR: track 0.00 -> 167.7 mm, vias 0 -> 4
- net VCC: track 0.00 -> 148.9 mm, vias 0 -> 3
- net /RC20: track 0.00 -> 138.5 mm
- net /RA13: track 0.00 -> 136.3 mm
- net /RC21: track 0.00 -> 133.2 mm
- net /RC26: track 0.00 -> 130.5 mm
- net /RA12: track 0.00 -> 125.1 mm, vias 0 -> 1
- net /RD2: track 0.00 -> 122.7 mm, vias 0 -> 2
- net /RD4: track 0.00 -> 119.4 mm, vias 0 -> 2
- net /RA11: track 0.00 -> 118.4 mm, vias 0 -> 1
- net /RD1: track 0.00 -> 118.0 mm, vias 0 -> 2
- net /RD6: track 0.00 -> 116.3 mm, vias 0 -> 2
- net /RA8: track 0.00 -> 114.0 mm, vias 0 -> 1
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
Commit message: updates for orders
Parts:
- added R4: R, Resistors_SMD:R_0805_HandSoldering, B.Cu at (137.4, 108.0)
- added R5: R, Resistors_SMD:R_0805_HandSoldering, B.Cu at (140.4, 108.0)
- added U7: 74HC04, Housings_SOIC:SOIC-14_3.9x8.7mm_Pitch1.27mm, F.Cu at (112.6, 117.9)
Connections:
- C1 pad 1: /3V3 -> VCC
- C2 pad 1: /3V3 -> VCC
- C3 pad 1: /3V3 -> VCC
- C4 pad 1: /3V3 -> VCC
- C5 pad 1: /3V3 -> VCC
- C6 pad 1: /3V3 -> VCC
- C7 pad 1: VCC -> /5V0
- J1 pad 1: /3V3 -> VCC
- J1 pad 17: /3V3 -> VCC
- J1 pad 2: VCC -> /5V0
- J1 pad 22: /DAT_DIR -> /RC25
- J1 pad 4: VCC -> /5V0
- J1 pad 40: /RC21 -> /DAT_DIR
- J2 pad 1: /3V3 -> VCC
- J2 pad 17: /3V3 -> VCC
- J2 pad 2: VCC -> /5V0
- J2 pad 22: /DAT_DIR -> /RC25
- J2 pad 4: VCC -> /5V0
- J2 pad 40: /RC21 -> /DAT_DIR
- P1 pad 25: VCC -> /5V0
- R1 pad 1: /3V3 -> VCC
- R2 pad 1: /3V3 -> VCC
- R3 pad 1: /3V3 -> VCC
- U1 pad 1: VCC -> /5V0
- U1 pad 22: /PH1 -> /nATN
- U1 pad 23: /3V3 -> VCC
- U1 pad 24: /3V3 -> VCC
- U2 pad 11: /RC18 -> /RC24
- U2 pad 5: /DAT_DIR -> /RC25
- U3 pad 1: /PH0 -> /ATN
- U3 pad 19: /PH0 -> /ATN
- U3 pad 20: /3V3 -> VCC
- U4 pad 1: /PH0 -> /ATN
- U4 pad 19: /PH0 -> /ATN
- U4 pad 20: /3V3 -> VCC
- U5 pad 20: /3V3 -> VCC
- U5 pad 3: /RC21 -> /RC18
Routing:
- net /3V3: track 203.1 -> 0.00 mm, vias 4 -> 0
- net /5V0: track 0.00 -> 133.9 mm, vias 0 -> 1
- net /RC21: track 133.2 -> 0.00 mm
- net VCC: track 148.9 -> 252.1 mm, vias 3 -> 4
- net /ATN: track 0.00 -> 98.8 mm, vias 0 -> 3
- net /RC25: track 0.00 -> 91.8 mm, vias 0 -> 2
- net /RW: track 25.7 -> 64.3 mm, vias 1 -> 2
- net /RC20: track 138.5 -> 102.6 mm, vias 0 -> 1
- net /PH0: track 65.4 -> 30.2 mm, vias 3 -> 0
- net /RA13: track 136.3 -> 106.8 mm, vias 0 -> 3
- net /nATN: track 0.00 -> 28.8 mm, vias 0 -> 1
- net /RA8: track 114.0 -> 88.4 mm
- net /DAT_DIR: track 167.7 -> 143.6 mm, vias 4 -> 2
- net /SLTSL: track 98.2 -> 74.5 mm, vias 1 -> 3
- net /RC27: track 64.6 -> 87.6 mm
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