File: rpmcv5/rpmcv4.kicad_pcb (KiCad board)
At the start: 2 copper layers, 85.1 x 81.3 mm, 38 parts, among them J1 RPi_GPIO, P1 CONN_02X25, P2 CONN_02X25, U1 74LS373, U2 74LS373, U3 74HC244, U4 74LS373, U5 LVC4245

Commit message: PRMC V5 and RPIAPPLE V1 updated
Parts:
- added U6: 74HC04, Housings_SOIC:SOIC-14_3.9x8.7mm_Pitch1.27mm, F.Cu at (206.0, 73.5)
- added U7: 74LS08, Housings_SOIC:SOIC-14_3.9x8.7mm_Pitch1.27mm, F.Cu at (197.1, 73.7)
- R10, R11, R12, R13, R14, U1, U2, U3, U4, U5: moved to B.Cu
- moved R14 66.7 mm to (201.4, 82.5), turned to 180 degrees
- moved R12 42.5 mm to (194.1, 106.2), turned to 270 degrees
- moved R10 30.2 mm to (148.3, 120.1), turned to 270 degrees
- moved R13 29.9 mm to (191.5, 120.0), turned to 270 degrees
- moved R11 24.0 mm to (194.1, 120.0), turned to 270 degrees
- moved G2 2.25 mm to (176.0, 73.5)
- moved G1 1.90 mm to (157.2, 73.8)
- moved U3 0.52 mm to (187.5, 73.4)
- moved U2 0.40 mm to (172.5, 73.4)
- moved U4 0.40 mm to (202.3, 73.5), turned to 270 degrees
- moved U1 0.40 mm to (140.0, 73.0), turned to 270 degrees
- turned U5 to 180 degrees
Connections:
- J1 pad 15: /RC22 -> /CAPS
- J1 pad 17: +3V3 -> +5V
- J1 pad 18: /RC24 -> /INT
- J1 pad 36: /RA16 -> /RC16
- J1 pad 37: /RC26 -> /BUSDIR
- J1 pad 40: /RC21 -> /HAN
- P1 pad 44: /RC24 -> /RC27
- P1 pad 7: /WAIT -> /RC25
- P2 pad 44: /RC24 -> /RC27
- P2 pad 7: /WAIT -> /RC25
- R1 pad 1: +3V3 -> /V3.3
- R10 pad 1: +3V3 -> /RC27
- R10 pad 2: /RC24 -> +3V3
- R11 pad 1: /RC22 -> /INT
- R11 pad 2: /INT -> +3V3
- R12 pad 1: /RC23 -> /RC25
- R12 pad 2: /WAIT -> +3V3
- R13 pad 1: GND -> /BUSDIR
- R13 pad 2: /RC22 -> +3V3
- R2 pad 1: +3V3 -> /V3.3
- R3 pad 1: +3V3 -> /V3.3
- R4 pad 1: +3V3 -> /V3.3
- R5 pad 1: +3V3 -> /V3.3
- R6 pad 1: +3V3 -> /V3.3
- R7 pad 1: +3V3 -> /V3.3
- R8 pad 1: +3V3 -> /V3.3
- R9 pad 1: +3V3 -> /V3.3
- U1 pad 20: +3V3 -> +5V
- U2 pad 20: +3V3 -> +5V
- U3 pad 18: /SLTSL3 -> Net-(U3-Pad18)
- U3 pad 2: /RC21 -> Net-(U3-Pad2)
- U4 pad 20: +3V3 -> +5V
- U5 pad 23: +3V3 -> +5V
Routing:
- net GND: track 0.00 -> 249.3 mm, vias 0 -> 2
- net +5V: track 0.00 -> 172.5 mm, vias 0 -> 4
- net /CAPS: track 15.1 -> 135.6 mm
- net /BUSDIR: track 0.00 -> 114.5 mm, vias 0 -> 1
- net +3V3: track 69.6 -> 182.0 mm, vias 0 -> 2
- net /A15: track 0.00 -> 110.1 mm
- net /RA12: track 0.00 -> 104.9 mm, vias 0 -> 2
- net /WR: track 0.00 -> 102.8 mm, vias 0 -> 2
- net /CLK: track 0.00 -> 101.5 mm, vias 0 -> 1
- net /RC27: track 0.00 -> 99.4 mm, vias 0 -> 2
- net /PWR: track 0.00 -> 98.2 mm
- net /RA14: track 0.00 -> 97.9 mm, vias 0 -> 2
- net /RA13: track 0.00 -> 97.0 mm, vias 0 -> 3
- net /RA15: track 0.00 -> 96.7 mm, vias 0 -> 2
- net /RA11: track 0.00 -> 88.6 mm, vias 0 -> 2
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Other:
- outline, holes or cut-outs redrawn
- board text added: "2018.4.30"
- board text added: "RPMC V5"
- board text removed: "2018.1.19"
- board text removed: "RPMC V4"

Commit message: SPC/APPLE/RPMC/RPMP updated for PCB order
Parts:
- removed R14: R, Resistors_SMD:R_0805_HandSoldering
Routing:
- net /RC23: track 35.4 -> 20.2 mm, vias 2 -> 1
Other:
- board text added: "74HC04"
- board text added: "74HC08"
- board text added: "74HC244"
- board text added: "74LVC4245"
- board text removed: "74HC245"
Changed lines of the file:
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@@
 (kicad_pcb (version 4) (host pcbnew 4.0.7)
   (general
-    (links 205)
+    (links 203)
     (no_connects 0)
     (area 128.829999 50.724999 214.070001 132.155001)
     (thickness 1.6)
-    (drawings 40)
-    (tracks 1312)
+    (drawings 47)
+    (tracks 1302)
     (zones 0)
-    (modules 40)
+    (modules 39)
     (nets 100)
   )
@@
     )
   )
-  (module Resistors_SMD:R_0805_HandSoldering (layer B.Cu)
-    (at 201.422 82.55 180)
-    (descr "Resistor SMD 0805, hand soldering")
-    (tags "resistor 0805")
-    (attr smd)
-    (fp_text reference R14 (at 0 1.7 180) (layer B.SilkS)
-      (effects (font (size 1 1) (thickness 0.15)) (justify mirror))
-    )
-    (fp_text value R (at 0 -1.75 180) (layer B.Fab)
-      (effects (font (size 1 1) (thickness 0.15)) (justify mirror))
-    )
-    (fp_text user %R (at 0 0 180) (layer B.Fab)
-      (effects (font (size 0.5 0.5) (thickness 0.075)) (justify mirror))
-    )
-    (fp_line (start -1 -0.62) (end -1 0.62) (layer B.Fab) (width 0.1))
-    (fp_line (start 1 -0.62) (end -1 -0.62) (layer B.Fab) (width 0.1))
-    (fp_line (start 1 0.62) (end 1 -0.62) (layer B.Fab) (width 0.1))
-    (fp_line (start -1 0.62) (end 1 0.62) (layer B.Fab) (width 0.1))
-    (fp_line (start 0.6 -0.88) (end -0.6 -0.88) (layer B.SilkS) (width 0.12))
-    (fp_line (start -0.6 0.88) (end 0.6 0.88) (layer B.SilkS) (width 0.12))
-    (fp_line (start -2.35 0.9) (end 2.35 0.9) (layer B.CrtYd) (width 0.05))
-    (fp_line (start -2.35 0.9) (end -2.35 -0.9) (layer B.CrtYd) (width 0.05))
-    (fp_line (start 2.35 -0.9) (end 2.35 0.9) (layer B.CrtYd) (width 0.05))
-    (fp_line (start 2.35 -0.9) (end -2.35 -0.9) (layer B.CrtYd) (width 0.05))
-    (pad 1 smd rect (at -1.35 0 180) (size 1.5 1.3) (layers B.Cu B.Paste B.Mask)
-      (net 1 GND))
-    (pad 2 smd rect (at 1.35 0 180) (size 1.5 1.3) (layers B.Cu B.Paste B.Mask)
-      (net 84 /RC23))
-    (model ${KISYS3DMOD}/Resistors_SMD.3dshapes/R_0805.wrl
-      (at (xyz 0 0 0))
-      (scale (xyz 1 1 1))
-      (rotate (xyz 0 0 0))
-    )
-  )
   (module Housings_SOIC:SOIC-20W_7.5x12.8mm_Pitch1.27mm (layer B.Cu)
     (at 139.954 73.024 270)
@@
     )
   )
+  (gr_circle (center 204.7621 69.7865) (end 205.0161 69.6595) (layer F.SilkS) (width 0.2))
+  (gr_circle (center 196.0245 69.9262) (end 196.2785 69.7992) (layer F.SilkS) (width 0.2))
+  (gr_text 74HC04 (at 205.8162 73.6219 270) (layer F.SilkS)
+    (effects (font (size 1.5 1.5) (thickness 0.3)))
+  )
+  (gr_text 74HC08 (at 197.2564 73.7743 270) (layer F.SilkS)
+    (effects (font (size 1.5 1.5) (thickness 0.3)))
+  )
+  (gr_circle (center 134.2898 70.2056) (end 134.5438 70.3326) (layer B.SilkS) (width 0.2))
+  (gr_circle (center 162.9664 74.93) (end 163.2204 75.057) (layer B.SilkS) (width 0.2))
+  (gr_circle (center 166.8018 70.5612) (end 167.0558 70.6882) (layer B.SilkS) (width 0.2))
+  (gr_circle (center 196.5198 70.6374) (end 196.7738 70.7644) (layer B.SilkS) (width 0.2))
   (gr_arc (start 148.59 52.07) (end 147.32 52.07) (angle 90) (layer Edge.Cuts) (width 0.15))
   (gr_arc (start 212.725 52.07) (end 212.725 50.8) (angle 90) (layer Edge.Cuts) (width 0.15))
@@
   )
   (gr_circle (center 198.755 73.787) (end 199.009 73.914) (layer B.SilkS) (width 0.2))
-  (gr_circle (center 182.245 73.533) (end 182.499 73.66) (layer B.SilkS) (width 0.2))
+  (gr_circle (center 181.7624 70.6628) (end 182.0164 70.7898) (layer B.SilkS) (width 0.2))
   (gr_circle (center 177.165 78.613) (end 177.419 78.74) (layer B.SilkS) (width 0.2))
-  (gr_circle (center 160.655 78.74) (end 160.909 78.867) (layer B.SilkS) (width 0.2))
-  (gr_text 74HC373 (at 171.45 76.2) (layer B.SilkS)
-    (effects (font (size 1.5 1.5) (thickness 0.375)) (justify mirror))
+  (gr_text 74HC373 (at 172.466 73.279 180) (layer B.SilkS)
+    (effects (font (size 1.5 1.5) (thickness 0.3)) (justify mirror))
   )
-  (gr_text 74HC373 (at 154.94 76.2) (layer B.SilkS)
+  (gr_text 74LVC4245 (at 156.1338 73.3552) (layer B.SilkS)
     (effects (font (size 1.5 1.5) (thickness 0.37)) (justify mirror))
   )
-  (gr_text 74HC245 (at 138.43 76.2) (layer B.SilkS)
-    (effects (font (size 1.5 1.5) (thickness 0.2)) (justify mirror))
+  (gr_text 74HC373 (at 139.954 73.1012 180) (layer B.SilkS)
+    (effects (font (size 1.5 1.5) (thickness 0.3)) (justify mirror))
   )
-  (gr_text 74HC245 (at 187.96 76.2) (layer B.SilkS)
+  (gr_text 74HC244 (at 187.4266 73.4314 180) (layer B.SilkS)
     (effects (font (size 1.5 1.5) (thickness 0.2)) (justify mirror))
   )
-  (gr_text 74HC245 (at 204.47 76.2) (layer B.SilkS)
-    (effects (font (size 1.5 1.5) (thickness 0.2)) (justify mirror))
+  (gr_text 74HC373 (at 202.5777 73.3933 180) (layer B.SilkS)
+    (effects (font (size 1.5 1.5) (thickness 0.3)) (justify mirror))
   )
   (gr_circle (center 132.715 73.533) (end 132.969 73.66) (layer B.SilkS) (width 0.2))
@@
   (segment (start 197.866 79.5323) (end 195.4376 81.9607) (width 0.25) (layer B.Cu) (net 24))
   (segment (start 197.866 78.232) (end 197.866 79.5323) (width 0.25) (layer B.Cu) (net 24))
+  (segment (start 202.946 78.232) (end 202.946 79.5323) (width 0.25) (layer B.Cu) (net 25))
+  (segment (start 200.8823 80.9648) (end 199.8029 80.9648) (width 0.25) (layer B.Cu) (net 25))
+  (segment (start 202.946 79.5323) (end 202.31241 79.5323) (width 0.25) (layer B.Cu) (net 25))
+  (segment (start 202.31241 79.5323) (end 200.8823 80.96241) (width 0.25) (layer B.Cu) (net 25))
+  (segment (start 200.8823 80.96241) (end 200.8823 80.9648) (width 0.25) (layer B.Cu) (net 25))
   (via (at 162.0126 79.4407) (size 0.6) (layers F.Cu B.Cu) (net 25))
   (via (at 199.8029 80.9648) (size 0.6) (layers F.Cu B.Cu) (net 25))
@@
   (segment (start 195.3872 80.9648) (end 199.8029 80.9648) (width 0.25) (layer F.Cu) (net 25))
   (segment (start 186.436 89.916) (end 195.3872 80.9648) (width 0.25) (layer F.Cu) (net 25))
-  (segment (start 202.3148 79.5323) (end 202.946 79.5323) (width 0.25) (layer B.Cu) (net 25))
-  (segment (start 201.3967 80.4504) (end 202.3148 79.5323) (width 0.25) (layer B.Cu) (net 25))
-  (segment (start 200.3173 80.4504) (end 201.3967 80.4504) (width 0.25) (layer B.Cu) (net 25))
-  (segment (start 199.8029 80.9648) (end 200.3173 80.4504) (width 0.25) (layer B.Cu) (net 25))
-  (segment (start 202.946 78.232) (end 202.946 79.5323) (width 0.25) (layer B.Cu) (net 25))
   (via (at 203.7452 87.3188) (size 0.6) (layers F.Cu B.Cu) (net 26))
   (segment (start 187.5472 114.5298) (end 186.436 115.641) (width 0.25) (layer B.Cu) (net 26))
@@
   (segment (start 189.1567 55.7276) (end 189.1567 56.095) (width 0.25) (layer F.Cu) (net 83))
   (via (at 193.0865 74.93) (size 0.6) (layers F.Cu B.Cu) (net 84))
-  (via (at 200.633 81.0843) (size 0.6) (layers F.Cu B.Cu) (net 84))
   (segment (start 194.437 74.93) (end 193.3617 74.93) (width 0.25) (layer F.Cu) (net 84))
   (segment (start 187.792 58.2676) (end 187.792 59.4429) (width 0.25) (layer B.Cu) (net 84))
-  (segment (start 200.072 82.55) (end 201.1473 82.55) (width 0.25) (layer B.Cu) (net 84))
   (segment (start 193.3617 74.93) (end 193.0865 74.93) (width 0.25) (layer F.Cu) (net 84))
-  (segment (start 201.1473 81.5986) (end 200.633 81.0843) (width 0.25) (layer B.Cu) (net 84))
-  (segment (start 201.1473 82.55) (end 201.1473 81.5986) (width 0.25) (layer B.Cu) (net 84))
-  (segment (start 200.633 80.9105) (end 200.633 81.0843) (width 0.25) (layer F.Cu) (net 84))
-  (segment (start 199.62 79.8975) (end 200.633 80.9105) (width 0.25) (layer F.Cu) (net 84))
-  (segment (start 194.6986 79.8975) (end 199.62 79.8975) (width 0.25) (layer F.Cu) (net 84))
-  (segment (start 192.9114 78.1103) (end 194.6986 79.8975) (width 0.25) (layer F.Cu) (net 84))
-  (segment (start 192.9114 75.3803) (end 192.9114 78.1103) (width 0.25) (layer F.Cu) (net 84))
-  (segment (start 193.3617 74.93) (end 192.9114 75.3803) (width 0.25) (layer F.Cu) (net 84))
   (segment (start 190.0016 71.8451) (end 193.0865 74.93) (width 0.25) (layer B.Cu) (net 84))
   (segment (start 190.0016 63.2618) (end 190.0016 71.8451) (width 0.25) (layer B.Cu) (net 84))

Commit message: updates for orders
Connections:
- U5 pad 23: +5V -> +3V3
Routing:
- net +5V: track 172.5 -> 165.0 mm
- net +3V3: track 182.0 -> 185.8 mm
