File: rpmcv5/rpmcv4.sch (KiCad schematic (older format))
At the start: 31 parts, among them J1 RPi_GPIO, P1 CONN_02X25, P2 CONN_02X25, U1 74LS373, U2 74LS373, U3 74HC244, U4 74LS373, U5 LVC4245

Commit message: PRMC V5 and RPIAPPLE V1 updated
Parts:
- removed R14: R, Resistors_SMD:R_0805_HandSoldering, symbol R
- added U6: 74HC04, Housings_SOIC:SOIC-14_3.9x8.7mm_Pitch1.27mm, symbol 74HC04
- added U7: 74LS08, Housings_SOIC:SOIC-14_3.9x8.7mm_Pitch1.27mm, symbol 74LS08
Connections:
- net labels added: 3V3, nPWR, nSLTSL3
- net labels removed: RA16
- wire segments 271 -> 281
- no-connect marks 15 -> 16
Other:
- note added: "2018.4.30"
- note added: "RPMC V5 with 74HC373 and 74LVC4245"
- note removed: "2017.12.29"
- note removed: "RPMC V4 with 74HC373 and 74HC245"

Commit message: updates for orders
Changed lines of the file:
@@
 LIBS:IC_raspberry
 LIBS:msx_slot
-LIBS:rpmcv4-cache
 EELAYER 25 0
 EELAYER END
@@
 3V3
 $Comp
-L +5V #PWR3
+L +5V #PWR01
 U 1 1 5A435798
 P 3500 4050
-F 0 "#PWR3" H 3500 3900 50  0001 C CNN
+F 0 "#PWR01" H 3500 3900 50  0001 C CNN
 F 1 "+5V" H 3500 4190 50  0000 C CNN
 F 2 "" H 3500 4050 50  0000 C CNN
@@
 	3500 4050 3500 4450
 $Comp
-L GND #PWR1
+L GND #PWR02
 U 1 1 5A4358D3
 P 655 6410
-F 0 "#PWR1" H 655 6160 50  0001 C CNN
+F 0 "#PWR02" H 655 6160 50  0001 C CNN
 F 1 "GND" H 655 6260 50  0000 C CNN
 F 2 "" H 655 6410 50  0000 C CNN
@@
 GND
 $Comp
-L +3.3V #PWR2
+L +3.3V #PWR03
 U 1 1 5A43A975
 P 800 4250
-F 0 "#PWR2" H 800 4100 50  0001 C CNN
+F 0 "#PWR03" H 800 4100 50  0001 C CNN
 F 1 "+3.3V" H 800 4390 50  0000 C CNN
 F 2 "" H 800 4250 50  0000 C CNN
@@
 $EndComp
 $Comp
-L GND #PWR5
+L GND #PWR04
 U 1 1 5A446BD1
 P 10800 3200
-F 0 "#PWR5" H 10800 2950 50  0001 C CNN
+F 0 "#PWR04" H 10800 2950 50  0001 C CNN
 F 1 "GND" H 10800 3050 50  0000 C CNN
 F 2 "" H 10800 3200 50  0001 C CNN
@@
 Connection ~ 655  5550
 $Comp
-L GND #PWR4
+L GND #PWR05
 U 1 1 5A5D9C37
 P 3655 6420
-F 0 "#PWR4" H 3655 6170 50  0001 C CNN
+F 0 "#PWR05" H 3655 6170 50  0001 C CNN
 F 1 "GND" H 3655 6270 50  0000 C CNN
 F 2 "" H 3655 6420 50  0000 C CNN
@@
 Wire Wire Line
 	6650 5450 7050 5450
-Text Label 6800 5450 0    60   ~ 0
-VCC
 Wire Wire Line
 	6650 5350 7050 5350
@@
 Text Label 6070 7460 0    60   ~ 0
 nPWR
+Text Label 6805 5450 0    60   ~ 0
+3V3
 $EndSCHEMATC
