File: rpispcv4/rpspc.sch (KiCad schematic (older format))
At the start: 5 parts, among them J1 RPi_GPIO, J2 Conn_02x17_Top_Bottom, J3 RPi_GPIO, U1 LVC4245, U2 74HC244

Commit message: SPC/APPLE/RPMC/RPMP updated for PCB order
Connections:
- wire segments 142 -> 143
Changed lines of the file:
@@
 LIBS:IC_raspberry
 LIBS:msx_slot
+LIBS:rpspc-cache
 EELAYER 25 0
 EELAYER END
@@
 Wire Wire Line
 	6895 2220 6245 2220
+Text Label 6395 2320 0    60   ~ 0
+VCC
+Wire Wire Line
+	6895 2320 6245 2320
 $EndSCHEMATC

Commit message: update for 74LVC2425 package
Parts:
- U1: footprint SMD_Packages:SOIC-24 -> Housings_SOIC:SOIC-24W_7.5x15.4mm_Pitch1.27mm
Changed lines of the file:
@@
 F 0 "U1" H 5545 3470 60  0000 C CNN
 F 1 "LVC4245" H 5595 2920 60  0000 C CNN
-F 2 "SMD_Packages:SOIC-24" H 5745 3370 60  0001 C CNN
+F 2 "Housings_SOIC:SOIC-24W_7.5x15.4mm_Pitch1.27mm" H 5745 3370 60  0001 C CNN
 F 3 "" H 5745 3370 60  0001 C CNN
 	1    5595 2770
