File: rpmcv7/_saved_rpmcv4.sch (KiCad schematic (older format))
At the start: 32 parts, among them J1 RPi_GPIO, P1 CONN_02X25, P2 CONN_02X25, U1 74LS373, U2 74LS373, U3 74HC244, U4 74LS373, U5 LVC4245, U6 74HC04, U7 74LS08

Commit message: update for 74LVC2425 package
Parts:
- added unit 3 of U6
- added unit 4 of U6
- added unit 5 of U6
- added unit 6 of U6
- added unit 3 of U7
- added unit 4 of U7
- U5: footprint SMD_Packages:SOIC-24 -> Housings_SOIC:SOIC-24W_7.5x15.4mm_Pitch1.27mm
Connections:
- net labels added: SLTSL2, nA14, nA15, nCS1, nCS12, nCS2
- net labels removed: nSLTSL3
- wire segments 281 -> 299
- no-connect marks 16 -> 12
Other:
- note added: "RPMC V7 with 74HC373 and 74LVC4245"
- note removed: "RPMC V5 with 74HC373 and 74LVC4245"
