File: rpmpv8/rpmpv1.kicad_pcb (KiCad board)
At the start: 2 copper layers, 90.4 x 64.4 mm, 30 parts, among them J1 RPi_GPIO, J2 RPi_GPIO, P1 CONN_02X25, U1 74HC244, U2 74HC04, U3 74HC244, U4 74HC244, U5 74LS07, U6 74LS08, U7 LVC4245

Commit message: RPMPV8 updated
Parts:
- U7: footprint MSX:SOIC-24@ -> Housings_SOIC:SOIC-24W_7.5x15.4mm_Pitch1.27mm
- moved U7 0.15 mm to (141.6, 93.1), turned to 90 degrees
Connections:
- J1 pad 40: /ATN -> /RC21
- J2 pad 40: /ATN -> /RC21
- U1 pad 1: GND -> /nRATN
- U1 pad 19: GND -> /nRATN
- U2 pad 11: /RC25 -> /nDIR
- U2 pad 8: /DAT_EN -> /nRC21
- U2 pad 9: /nDAT_EN -> /RC21
- U3 pad 12: /RD5 -> /RA13
- U3 pad 14: /RD4 -> /RA12
- U3 pad 16: /RD7 -> /RA15
- U3 pad 18: /RD6 -> /RA14
- U3 pad 3: /RD2 -> /RA10
- U3 pad 5: /RD3 -> /RA11
- U3 pad 7: /RD0 -> /RA8
- U3 pad 9: /RD1 -> /RA9
- U4 pad 16: Net-(U4-Pad16) -> /RC27
- U4 pad 5: Net-(U4-Pad5) -> /RC26
- U6 pad 1: /MREQ -> /DAT_EN0
- U6 pad 11: (no net) -> /nDIR
- U6 pad 12: (no net) -> /WR
- U6 pad 13: (no net) -> /RC25
- U6 pad 2: /IORQ -> /nRC21
- U6 pad 3: /nATN -> /DAT_EN
- U6 pad 4: /ATN -> /SLTSL
- U6 pad 5: /RATN -> /IORQ
- U6 pad 6: /nDAT_EN -> /DAT_EN0
Routing:
- net GND: track 0.00 -> 343.2 mm, vias 0 -> 4
- net +3V3: track 0.00 -> 220.7 mm, vias 0 -> 5
- net +5V: track 0.00 -> 176.0 mm, vias 0 -> 2
- net /RA13: track 0.00 -> 130.7 mm, vias 0 -> 1
- net /RC17: track 0.00 -> 126.0 mm
- net /RC25: track 0.00 -> 118.4 mm
- net /RA9: track 0.00 -> 109.4 mm, vias 0 -> 1
- net /IORQ: track 0.00 -> 108.0 mm, vias 0 -> 2
- net /RA8: track 0.00 -> 104.2 mm, vias 0 -> 1
- net /RA14: track 0.00 -> 97.5 mm
- net /DAT_DIR: track 0.00 -> 95.3 mm, vias 0 -> 3
- net /RA15: track 0.00 -> 92.6 mm, vias 0 -> 2
- net /RC18: track 0.00 -> 92.3 mm
- net /RATN: track 0.00 -> 89.0 mm, vias 0 -> 1
- net /nRATN: track 0.00 -> 88.4 mm
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Other:
- board text added: "Rraspberry Pi extension Ver. 1.2"
- board text removed: "Rraspberry Pi extension Ver. 1.1"

Commit message: PCB ordered RPMPV8, RPMCV8, RPISPCV5
Other:
- board text added: "2018.06.27"
- board text removed: "2018.05.18"
