File: rpmcv9/_autosave-rpmcv4.kicad_pcb (KiCad board)
At the start: 2 copper layers, 98.2 x 81.9 mm, 33 parts, among them J1 RPi_GPIO, P1 CONN_02X25, P2 CONN_02X25, U1 74LS373, U2 74LS373, U3 74HC595, U4 74LS373, U5 LVC4245, U7 74LS08

Commit message: lastest update
Parts:
- added D7: LED, LEDs:LED_D3.0mm, F.Cu at (144.8, 130.8)
- added D8: LED, LEDs:LED_D3.0mm, F.Cu at (182.9, 130.8)
- added R10: R, Resistors_SMD:R_0603_HandSoldering, B.Cu at (146.1, 127.6)
- added R11: R, Resistors_SMD:R_0603_HandSoldering, B.Cu at (184.2, 127.6)
- moved GMSX 5.99 mm to (162.5, 130.5)
- moved R4 3.58 mm to (139.7, 127.6)
- moved D4 3.31 mm to (138.4, 130.8)
- moved R5 2.04 mm to (190.5, 127.6)
- moved D5 1.80 mm to (189.2, 130.8)
- moved D3 1.55 mm to (132.1, 130.8)
- moved R3 1.33 mm to (133.3, 127.6)
- moved R2 0.77 mm to (196.8, 127.6)
- moved R6 0.63 mm to (127.0, 127.6)
- moved D2 0.57 mm to (195.6, 130.8)
- moved D6 0.36 mm to (125.7, 130.8)
- moved D1 0.36 mm to (201.9, 130.8)
- moved R1 0.13 mm to (203.2, 127.6)
- renumbered G*** to GMSX
Routing:
- net /RC26: track 73.2 -> 100.5 mm, vias 0 -> 1
- net GND: track 365.2 -> 392.4 mm, vias 2 -> 1
- net Net-(D8-Pad2): track 0.00 -> 25.6 mm
- net /RA10: track 72.9 -> 52.2 mm
- net /RC16: track 27.7 -> 47.2 mm, vias 3 -> 1
- net Net-(D7-Pad2): track 0.00 -> 17.5 mm
- net /RD7: track 51.4 -> 67.2 mm, vias 2 -> 0
- net /RD4: track 85.3 -> 70.1 mm, vias 0 -> 2
- net /RD6: track 50.6 -> 65.5 mm
- net /RC23: track 93.3 -> 78.4 mm, vias 2 -> 0
- net Net-(D1-Pad1): track 13.3 -> 3.25 mm
- net /RC21: track 39.9 -> 31.2 mm, vias 0 -> 1
- net /RA13: track 57.3 -> 48.8 mm, vias 0 -> 2
- net /RD2: track 69.9 -> 78.0 mm, vias 1 -> 2
- net /A1: track 46.5 -> 54.1 mm, vias 1 -> 0
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Other:
- board text added: "opt1"
- board text added: "opt2"
