File: rpmcv9/rpmcv4.sch (KiCad schematic (older format))
At the start: 24 parts, among them J1 RPi_GPIO, P1 CONN_02X25, P2 CONN_02X25, U1 74LS373, U2 74LS373, U3 74HC595, U4 74LS373, U5 LVC4245, U7 74LS08

Commit message: RPMC V9 for real-like MSX machine
Other:
- note added: "RC16 LE_A\nRC17 LE_C\nRC18 LE_D\nRC19 RESET\nRC20 CLK\nRC21 DAT_DIR\nRC22 SRCLK\nRC23 RCLK\nRC24 INT\nRC25 WAIT\nRC26 SER\nRC27 SW1"
- note removed: "RC16 LE_A\nRC17 LE_C\nRC18 LE_D\nRC19 RESET\nRC20 CLK\nRC21 SER\nRC22 SRCLK\nRC23 RCLK\nRC24 INT\nRC25 WAIT\nRC26 SW1"
Changed lines of the file:
@@
 RD6
 Text Label 8320 3545 0    60   ~ 0
-WR
+RC21
 Text Label 8320 2645 0    60   ~ 0
 GND
@@
 3V3
 Text Label 6930 5230 0    60   ~ 0
-RC26
+RC27
 Text Label 8150 5230 0    60   ~ 0
 SW1
@@
 3V3
 Text Notes 4700 6890 0    60   ~ 0
-RC16   LE_A\nRC17   LE_C\nRC18   LE_D\nRC19   RESET\nRC20   CLK\nRC21   SER\nRC22   SRCLK\nRC23   RCLK\nRC24   INT\nRC25   WAIT\nRC26   SW1
+RC16   LE_A\nRC17   LE_C\nRC18   LE_D\nRC19   RESET\nRC20   CLK\nRC21   DAT_DIR\nRC22   SRCLK\nRC23   RCLK\nRC24   INT\nRC25   WAIT\nRC26   SER\nRC27   SW1
 $Comp
 L 74LS08 U7
@@
 RC22
 Text Label 3415 6860 0    60   ~ 0
-RC21
+RC26
 Wire Wire Line
 	2935 7010 2935 7220

Commit message: lastest update
Parts:
- added D7, D8: LED, LEDs:LED_D3.0mm, symbol LED
- added R10, R11: R, Resistors_SMD:R_0603_HandSoldering, symbol R
Connections:
- wire segments 279 -> 289
- no-connect marks 7 -> 5
