File: rpemv1/rpmcv4.sch (KiCad schematic (older format))
At the start: 17 parts, among them J1 RPi_GPIO, J2 Conn_02x02_Odd_Even, J3 Conn_01x05_Male, U1 74LS373, U2 74LS373, U3 Z80CPU, U4 74LS373, U5 LVC4245, U6 74HC244

Commit message: many changes
Parts:
- added J4: RPi_GPIO, Socket_Strips:Socket_Strip_Straight_2x20_Pitch2.54mm, symbol RPi_GPIO
Connections:
- wire segments 207 -> 252
