File: rpiz80v4/msxbox.kicad_pcb (KiCad board)
At the start: 2 copper layers, 65 x 56.5 mm, 18 parts, among them J1 Raspberry_Pi_2_3, U1 Z80CPU, U2 74LS244, U3 74LS244, U4 LVC4245, U5 74LS244, U6 74LS244, U7 74LS05

Commit message: many changes
Parts:
- U2, U3, U5, U6: value 74LS244 -> 74HC244
- moved G*** 15.2 mm to (124.5, 71.1)
- moved R1 1.37 mm to (154.4, 78.2)
- moved D2 1.27 mm to (96.3, 71.0)
- moved D3 1.27 mm to (96.3, 78.2)
- moved R2 1.27 mm to (96.3, 71.0)
- moved R3 1.27 mm to (96.3, 78.2)
- moved D4 1.02 mm to (154.4, 71.1)
- moved R4 1.02 mm to (154.4, 71.1)
- moved D1 1.02 mm to (154.4, 77.9)
Connections:
- J1 pad 1: VCC -> /3V3
- J1 pad 17: VCC -> /3V3
- J1 pad 26: /RC7 -> /RD7
- U2 pad 1: GND -> /RATN
- U2 pad 11: /RC20 -> /A7
- U2 pad 12: /BUSRQ -> /RD3
- U2 pad 13: /RC16 -> /A6
- U2 pad 14: /NMI -> /RD2
- U2 pad 15: /RC17 -> /A5
- U2 pad 16: /INT -> /RD1
- U2 pad 17: Net-(U2-Pad17) -> /A4
- U2 pad 18: /WAIT -> /RD0
- U2 pad 19: GND -> /RATN
- U2 pad 2: /RC24 -> /A0
- U2 pad 20: VCC -> /3V3
- U2 pad 3: Net-(U2-Pad3) -> /RD4
- U2 pad 4: /RC23 -> /A1
- U2 pad 5: /DAT_DIR -> /RD5
- U2 pad 6: /RC25 -> /A2
- U2 pad 7: /RESET -> /RD6
- U2 pad 8: /RC26 -> /A3
- U2 pad 9: /CLK -> /RD7
- U3 pad 11: /A12 -> /A15
- U3 pad 13: /A13 -> /A14
- U3 pad 15: /A14 -> /A13
- U3 pad 17: /A15 -> /A12
- U3 pad 20: VCC -> /3V3
- U3 pad 3: /RA15 -> /RA12
- U3 pad 5: /RA14 -> /RA13
- U3 pad 7: /RA13 -> /RA14
- U3 pad 9: /RA12 -> /RA15
- U4 pad 23: VCC -> /3V3
- U4 pad 24: VCC -> /3V3
- U5 pad 11: RD -> Net-(U5-Pad11)
- U5 pad 12: /RC22 -> /BUSRQ
- U5 pad 13: WR -> /RC17
- U5 pad 14: /RC21 -> /NMI
- U5 pad 15: /M1 -> /RC16
- U5 pad 16: /RC18 -> /INT
- U5 pad 17: /RFSH -> /RC20
- U5 pad 18: /RC19 -> /WAIT
- U5 pad 19: /DAT_EN -> GND
- U5 pad 2: MERQ -> /RC24
- U5 pad 20: VCC -> +5V
- U5 pad 3: /RA15 -> /CLK
- U5 pad 4: IORQ -> /RC23
- U5 pad 5: /RA14 -> /RESET
- U5 pad 6: /HALT -> /RC25
- U5 pad 7: /RA13 -> /DAT_DIR
- U5 pad 8: /BUSACK -> /RC26
- U5 pad 9: /RA12 -> Net-(U5-Pad9)
- U6 pad 1: /RATN -> GND
- U6 pad 11: /A4 -> /RFSH
- U6 pad 12: /RD3 -> /RC22
- U6 pad 13: /A5 -> /M1
- U6 pad 14: /RD2 -> /RC21
- U6 pad 15: /A6 -> WR
- U6 pad 16: /RD1 -> /RC18
- U6 pad 17: /A7 -> RD
- U6 pad 18: /RD0 -> /RC19
- U6 pad 19: /RATN -> /DAT_EN
- U6 pad 2: /A0 -> MERQ
- U6 pad 20: VCC -> /3V3
- U6 pad 3: /RD7 -> /RA12
- U6 pad 4: /A1 -> IORQ
- U6 pad 5: /RD6 -> /RA13
- U6 pad 6: /A2 -> /HALT
- U6 pad 7: /RD5 -> /RA14
- U6 pad 8: /A3 -> /BUSACK
- U6 pad 9: /RD4 -> /RA15
Routing:
- net /3V3: track 0.00 -> 101.9 mm, vias 0 -> 3
- net MERQ: track 23.8 -> 107.7 mm
- net VCC: track 171.8 -> 112.7 mm, vias 4 -> 2
- net /RA12: track 85.7 -> 31.7 mm, vias 0 -> 1
- net /RC21: track 74.2 -> 28.3 mm
- net /M1: track 41.3 -> 87.2 mm, vias 2 -> 0
- net /RC20: track 113.9 -> 72.5 mm, vias 2 -> 1
- net /RA13: track 63.1 -> 24.0 mm, vias 2 -> 1
- net +5V: track 112.2 -> 76.6 mm, vias 0 -> 1
- net WR: track 45.7 -> 77.5 mm, vias 0 -> 2
- net /HALT: track 34.2 -> 64.8 mm
- net /RA14: track 87.2 -> 58.1 mm
- net /A5: track 44.9 -> 73.0 mm, vias 1 -> 0
- net IORQ: track 84.5 -> 111.3 mm
- net /A4: track 44.8 -> 69.2 mm, vias 1 -> 0
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Other:
- board text added: "2018.11.26"
- board text added: "Real Z80 Processor Engine V2.1 [Z80BOX]"
- board text removed: "2018.9.10"
- board text removed: "Real Z80 Processor Engine V2.0 [Z80BOX]"
