File: rpmcv2019-1/rpmcv4.kicad_pcb (KiCad board)
At the start: 2 copper layers, 99.3 x 81.9 mm, 34 parts, among them J1 RPi_GPIO, P1 CONN_02X25, P2 CONN_02X25, U1 74LS373, U2 74LS373, U3 74HC595, U4 74LS373, U5 LVC4245, U7 74LS08

Commit message: many changes
Connections:
- P1 pad 50: /+12V -> /-12V
- P2 pad 50: /+12V -> /-12V
Routing:
- net /-12V: track 0.00 -> 24.1 mm
- net /+12V: track 28.0 -> 24.1 mm
Changed lines of the file:
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@@
 (kicad_pcb (version 4) (host pcbnew 4.0.7)
   (general
-    (links 191)
+    (links 190)
     (no_connects 0)
     (area 111.254174 52.883999 210.720798 134.949001)
     (thickness 1.6)
     (drawings 59)
-    (tracks 1152)
+    (tracks 1155)
     (zones 0)
     (modules 34)
-    (nets 93)
+    (nets 94)
   )
   (page A4)
@@
   (net 91 "Net-(D8-Pad1)")
   (net 92 "Net-(D8-Pad2)")
+  (net 93 /-12V)
   (net_class Default "This is the default net class."
     (clearance 0.2)
@@
     (add_net +3V3)
     (add_net /+12V)
+    (add_net /-12V)
     (add_net /A0)
     (add_net /A1)
@@
       (net 51 /SNDIN))
     (pad 50 thru_hole circle (at -31.75 2.54) (size 1.524 1.524) (drill 0.777) (layers *.Cu *.Mask F.SilkS)
-      (net 50 /+12V))
+      (net 93 /-12V))
   )
   (module MSX:MSX_SLOT locked (layer F.Cu)
@@
       (net 51 /SNDIN))
     (pad 50 thru_hole circle (at -31.75 2.54) (size 1.524 1.524) (drill 0.777) (layers *.Cu *.Mask F.SilkS)
-      (net 50 /+12V))
+      (net 93 /-12V))
   )
   (module LEDs:LED_D3.0mm (layer F.Cu)
@@
   (segment (start 146.7442 116.9988) (end 146.7442 96.1072) (width 0.25) (layer B.Cu) (net 49))
   (segment (start 145.633 118.11) (end 146.7442 116.9988) (width 0.25) (layer B.Cu) (net 49))
-  (segment (start 135.473 118.11) (end 136.743 118.11) (width 0.25) (layer F.Cu) (net 50))
-  (segment (start 136.743 118.11) (end 138.013 118.11) (width 0.25) (layer F.Cu) (net 50))
-  (segment (start 135.473 94.996) (end 136.743 96.266) (width 0.25) (layer F.Cu) (net 50))
-  (segment (start 136.743 118.11) (end 136.743 96.266) (width 0.25) (layer F.Cu) (net 50))
-  (segment (start 136.743 96.266) (end 138.013 94.996) (width 0.25) (layer F.Cu) (net 50))
+  (segment (start 138.013 94.996) (end 138.013 109.819) (width 0.25) (layer B.Cu) (net 50))
+  (segment (start 139.192 116.931) (end 138.013 118.11) (width 0.25) (layer B.Cu) (net 50))
+  (segment (start 139.192 110.998) (end 139.192 116.931) (width 0.25) (layer B.Cu) (net 50))
+  (segment (start 138.013 109.819) (end 139.192 110.998) (width 0.25) (layer B.Cu) (net 50))
   (segment (start 134.3786 91.0104) (end 135.473 89.916) (width 0.25) (layer B.Cu) (net 51))
   (segment (start 134.3786 111.9356) (end 134.3786 91.0104) (width 0.25) (layer B.Cu) (net 51))
@@
   (segment (start 159.385 129.5053) (end 161.8811 132.0014) (width 0.25) (layer B.Cu) (net 92))
   (segment (start 159.385 128.43) (end 159.385 129.5053) (width 0.25) (layer B.Cu) (net 92))
+  (segment (start 135.473 94.996) (end 135.473 110.581) (width 0.25) (layer F.Cu) (net 93))
+  (segment (start 136.652 116.931) (end 135.473 118.11) (width 0.25) (layer F.Cu) (net 93))
+  (segment (start 136.652 111.76) (end 136.652 116.931) (width 0.25) (layer F.Cu) (net 93))
+  (segment (start 135.473 110.581) (end 136.652 111.76) (width 0.25) (layer F.Cu) (net 93))
   (zone (net 1) (net_name GND) (layer F.Cu) (hatch edge 0.508)
     (connect_pads (clearance 0.508))
