File: rpmcv2019-1/rpmcv4.sch (KiCad schematic (older format))
At the start: 25 parts, among them J1 RPi_GPIO, P1 CONN_02X25, P2 CONN_02X25, U1 74LS373, U2 74LS373, U3 74HC595, U4 74LS373, U5 LVC4245, U7 74LS08

Commit message: many changes
Connections:
- net labels added: -12V
Changed lines of the file:
@@
 SNDIN
 Text Label 10100 3345 0    60   ~ 0
-+12V
+-12V
 Text Label 10100 3245 0    60   ~ 0
 +12V
@@
 SNDIN
 Text Label 10095 6230 0    60   ~ 0
-+12V
+-12V
 Text Label 10095 6130 0    60   ~ 0
 +12V
