File: rompack/rompack.kicad_pcb (KiCad board)
At the start: 2 copper layers, 65.2 x 41.5 mm, 4 parts, among them P1 CONN_MSXSLOT, U1 28C256

Commit message: many changes
Parts:
- moved G*** 13.6 mm to (161.7, 91.3)
- moved U1 7.88 mm to (133.3, 98.8)
- moved G1 6.54 mm to (150.0, 91.1)
Connections:
- P1 pad 3: /SLTSL -> /CS12
- P1 pad 4: Net-(P1-Pad4) -> /SLTSL
- P1 pad 45: /5V0 -> VCC
- P1 pad 47: /5V0 -> VCC
- P1 pad 5: Net-(P1-Pad5) -> /WR0
- U1 pad 22: /RD -> /CS12
- U1 pad 27: Net-(U1-Pad27) -> /WR0
Routing:
- net /WR0: track 0.00 -> 55.3 mm
- net /CS12: track 0.00 -> 44.3 mm
- net VCC: track 0.00 -> 35.2 mm
- net /A14: track 56.9 -> 43.3 mm, vias 0 -> 1
- net /D7: track 55.4 -> 43.2 mm, vias 0 -> 1
- net /5V0: track 11.2 -> 0.00 mm
- net /A5: track 19.7 -> 10.6 mm
- net /A4: track 19.6 -> 11.1 mm, vias 1 -> 0
- net /A8: track 38.5 -> 30.0 mm, vias 1 -> 0
- net /A3: track 19.1 -> 11.0 mm
- net /A2: track 21.0 -> 13.2 mm
- net GND: track 57.2 -> 65.0 mm, vias 1 -> 0
- net /A10: track 39.5 -> 31.8 mm, vias 1 -> 0
- net /A1: track 20.7 -> 13.1 mm
- net /A0: track 23.2 -> 15.7 mm
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Other:
- board size 65.2 x 41.5 mm -> 65.2 x 35.6 mm
- board text added: "16KB/32KB ROMPACK"
- board text added: "2019.1.21"
- board text added: "28C256"
- board text added: "meeso.kim@gmail.com"
- board text removed: "2018.9.12"

Commit message: major updates for PCB
Parts:
- added R1: R, Resistors_SMD:R_0805_HandSoldering, B.Cu at (134.5, 87.6)
Routing:
- net VCC: track 35.2 -> 39.3 mm
- net /WR0: track 55.3 -> 59.3 mm
Other:
- board text added: "2019.2.20"
- board text removed: "2019.1.21"
Changed lines of the file:
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@@
 (kicad_pcb (version 4) (host pcbnew 4.0.7)
   (general
-    (links 31)
+    (links 33)
     (no_connects 0)
     (area 117.145999 76.899699 182.449136 112.649918)
     (thickness 1.6)
     (drawings 14)
-    (tracks 249)
+    (tracks 253)
     (zones 0)
-    (modules 4)
+    (modules 5)
     (nets 48)
   )
@@
       (xy 1.633829 -1.594475) (xy 1.687285 -1.5875) (xy 1.791864 -1.629393)) (layer B.SilkS) (width 0.01))
   )
+  (module Resistors_SMD:R_0805_HandSoldering (layer B.Cu)
+    (at 134.5438 87.5665 180)
+    (descr "Resistor SMD 0805, hand soldering")
+    (tags "resistor 0805")
+    (attr smd)
+    (fp_text reference R1 (at 0 1.7 180) (layer B.SilkS)
+      (effects (font (size 1 1) (thickness 0.15)) (justify mirror))
+    )
+    (fp_text value R (at 0 -1.75 180) (layer B.Fab)
+      (effects (font (size 1 1) (thickness 0.15)) (justify mirror))
+    )
+    (fp_text user %R (at 0 0 180) (layer B.Fab)
+      (effects (font (size 0.5 0.5) (thickness 0.075)) (justify mirror))
+    )
+    (fp_line (start -1 -0.62) (end -1 0.62) (layer B.Fab) (width 0.1))
+    (fp_line (start 1 -0.62) (end -1 -0.62) (layer B.Fab) (width 0.1))
+    (fp_line (start 1 0.62) (end 1 -0.62) (layer B.Fab) (width 0.1))
+    (fp_line (start -1 0.62) (end 1 0.62) (layer B.Fab) (width 0.1))
+    (fp_line (start 0.6 -0.88) (end -0.6 -0.88) (layer B.SilkS) (width 0.12))
+    (fp_line (start -0.6 0.88) (end 0.6 0.88) (layer B.SilkS) (width 0.12))
+    (fp_line (start -2.35 0.9) (end 2.35 0.9) (layer B.CrtYd) (width 0.05))
+    (fp_line (start -2.35 0.9) (end -2.35 -0.9) (layer B.CrtYd) (width 0.05))
+    (fp_line (start 2.35 -0.9) (end 2.35 0.9) (layer B.CrtYd) (width 0.05))
+    (fp_line (start 2.35 -0.9) (end -2.35 -0.9) (layer B.CrtYd) (width 0.05))
+    (pad 1 smd rect (at -1.35 0 180) (size 1.5 1.3) (layers B.Cu B.Paste B.Mask)
+      (net 46 /WR0))
+    (pad 2 smd rect (at 1.35 0 180) (size 1.5 1.3) (layers B.Cu B.Paste B.Mask)
+      (net 43 VCC))
+    (model ${KISYS3DMOD}/Resistors_SMD.3dshapes/R_0805.wrl
+      (at (xyz 0 0 0))
+      (scale (xyz 1 1 1))
+      (rotate (xyz 0 0 0))
+    )
+  )
   (dimension 42.292716 (width 0.3) (layer Eco1.User)
     (gr_text "42.293 mm" (at 190.131528 92.2044 89.48383577) (layer Eco1.User)
@@
     (effects (font (size 1.5 1.5) (thickness 0.3)))
   )
-  (gr_text "2019.1.21\n" (at 149.479 101.7778) (layer B.SilkS)
+  (gr_text "2019.2.20\n" (at 149.479 101.7778) (layer B.SilkS)
     (effects (font (size 2 2) (thickness 0.4)) (justify mirror))
   )
@@
   (segment (start 124.3608 108.1514) (end 124.3608 103.8261) (width 0.25) (layer F.Cu) (net 39))
   (segment (start 126.8958 107.6587) (end 126.8958 103.8334) (width 0.25) (layer F.Cu) (net 39))
+  (segment (start 133.1938 87.5665) (end 133.1938 83.7222) (width 0.25) (layer B.Cu) (net 43))
+  (segment (start 133.1938 83.7222) (end 133.35 83.566) (width 0.25) (layer B.Cu) (net 43))
   (segment (start 124.3608 93.599) (end 124.3838 93.599) (width 0.25) (layer B.Cu) (net 43))
   (segment (start 133.35 84.6328) (end 133.35 83.566) (width 0.25) (layer B.Cu) (net 43))
@@
   (segment (start 177.701 103.826) (end 159.3046 85.4296) (width 0.25) (layer B.Cu) (net 45))
   (segment (start 148.59 83.566) (end 149.7653 83.566) (width 0.25) (layer B.Cu) (net 45))
+  (segment (start 135.8938 87.5665) (end 135.8938 83.5698) (width 0.25) (layer B.Cu) (net 46))
+  (segment (start 135.8938 83.5698) (end 135.89 83.566) (width 0.25) (layer B.Cu) (net 46))
   (segment (start 135.89 83.566) (end 137.0653 83.566) (width 0.25) (layer B.Cu) (net 46))
   (segment (start 175.161 103.1646) (end 175.161 105.6578) (width 0.25) (layer B.Cu) (net 46))
