File: rompackwriter/rompack.kicad_pcb (KiCad board)
At the start: 2 copper layers, 76.2 x 22.9 mm, 2 parts, among them P1 CONN_MSXSLOT, U1 28C256

Commit message: major updates for PCB
Parts:
- added G***: LOGO, MSX:msxlogo, F.Cu at (116.1, 112.9)
- added G1: LOGO, MSX:srxg10, B.Cu at (115.4, 113.0)
- moved U1 0.90 mm to (181.5, 97.3)
Routing:
- net /D2: track 30.0 -> 21.3 mm
- net /D0: track 32.5 -> 25.9 mm
- net /D7: track 33.9 -> 37.1 mm
- net /A12: track 32.2 -> 34.8 mm, vias 1 -> 0
- net /D3: track 18.5 -> 20.5 mm
- net /A7: track 28.5 -> 26.5 mm
- net /CS12: track 17.4 -> 18.2 mm
- net GND: track 26.9 -> 26.2 mm
- net /D5: track 27.8 -> 28.4 mm
- net /A3: track 28.3 -> 27.7 mm
- net /A14: track 29.6 -> 28.9 mm
- net /A1: track 19.5 -> 18.9 mm
- net /D1: track 19.5 -> 18.9 mm
- net /WR0: track 12.2 -> 12.7 mm
- net /A4: track 34.6 -> 34.0 mm
Other:
- board text added: "2019.2.21"
- board text added: "28C256 ROMPACK WRITER"
- board text added: "meeso.kim@gmail.com"
- board text removed: "2019.1.21"
- board text removed: "MSX 28C256 Romwriter Socket"
