File: rpmcv2019-2/rpmcv4.kicad_pcb (KiCad board)
At the start: 2 copper layers, 97.7 x 56 mm, 13 parts, among them J1 RPi_GPIO, P1 CONN_02X25, U1 74LS373, U2 74LS373, U4 74LS373, U5 LVC4245, U7 74LS08

Commit message: major updates for PCB
Parts:
- added G***: LOGO, MSX:srxg, B.Cu at (203.8, 93.6)
- added G1: LOGO, MSX:raspberry_pi_logo, F.Cu at (172.1, 93.2)
- added G2: LOGO, MSX:msx_msx2_msx+logo, F.Cu at (193.8, 92.7)
- added REF1: MountingHole_2.5mm, Mounting_Holes:MountingHole_2.5mm, F.Cu at (119.2, 110.9)
- added REF2: MountingHole_2.5mm, Mounting_Holes:MountingHole_2.5mm, F.Cu at (119.2, 61.9)
- added REF3: MountingHole_2.5mm, Mounting_Holes:MountingHole_2.5mm, F.Cu at (177.1, 62.0)
- added REF4: MountingHole_2.5mm, Mounting_Holes:MountingHole_2.5mm, F.Cu at (209.5, 61.9)
- added REF5: MountingHole_2.5mm, Mounting_Holes:MountingHole_2.5mm, F.Cu at (177.2, 111.0)
- added REF6: MountingHole_2.5mm, Mounting_Holes:MountingHole_2.5mm, F.Cu at (209.8, 111.0)
- moved D1 2.79 mm to (182.8, 110.5)
- moved D2 2.79 mm to (191.7, 110.5)
- moved D3 2.79 mm to (200.6, 110.5)
- moved R2 2.79 mm to (193.0, 106.7)
- moved R3 2.79 mm to (201.9, 106.7)
- moved R1 2.79 mm to (184.1, 106.7)
Connections:
- P1 pad 10: (no net) -> /BUSDIR
- P1 pad 16: (no net) -> Net-(P1-Pad16)
- P1 pad 48: (no net) -> /+12V
- P1 pad 49: (no net) -> /SNDIN
- P1 pad 5: /M1 -> /WR_EXT
- P1 pad 50: (no net) -> /-12V
- P1 pad 6: (no net) -> /RFSH
- U4 pad 5: /M1 -> /WR_EXT
Routing:
- net GND: track 0.00 -> 233.2 mm, vias 0 -> 3
- net +5V: track 163.1 -> 116.6 mm, vias 5 -> 2
- net /RC25: track 71.2 -> 114.6 mm, vias 1 -> 0
- net /RD5: track 42.6 -> 68.8 mm, vias 2 -> 1
- net /RA8: track 86.1 -> 61.4 mm, vias 2 -> 3
- net /M1: track 87.3 -> 66.7 mm
- net /RC17: track 47.8 -> 67.4 mm
- net /WR_EXT: track 0.00 -> 18.0 mm
- net /A0: track 36.7 -> 21.4 mm, vias 0 -> 1
- net /RD4: track 38.8 -> 53.8 mm, vias 2 -> 1
- net /RC20: track 34.7 -> 19.9 mm
- net +3V3: track 76.1 -> 90.6 mm
- net /RD2: track 37.0 -> 49.6 mm, vias 2 -> 1
- net /RA11: track 74.4 -> 62.5 mm
- net /RC18: track 41.5 -> 30.2 mm, vias 0 -> 1
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Other:
- board text added: "2019.2.20"
- board text removed: "2019.01.23"
