File: rpmcv2019-2/rpmcv4.sch (KiCad schematic (older format))
At the start: 13 parts, among them J1 RPi_GPIO, P1 CONN_02X25, U1 74LS373, U2 74LS373, U4 74LS373, U5 LVC4245, U7 74LS08

Commit message: major updates for PCB
Other:
- note added: "RC16 LE_A\nRC17 LE_C\nRC18 LE_D\nRC19 RESET\nRC20 CLK\nRC21 DAT_DIR\nRC22 LED_CODE\nRC23 LED_CAPS\nRC24 INT\nRC25 WAIT\nRC26 LED_HAN\nRC27 SW1"
- note removed: "RC16 LE_A\nRC17 LE_C\nRC18 LE_D\nRC19 RESET\nRC20 CLK\nRC21 DAT_DIR\nRC22 LED_POWER\nRC23 LED_CAPS\nRC24 INT\nRC25 WAIT\nRC26 LED_HAN\nRC27 SW1"
Changed lines of the file:
@@
 3V3
 Text Notes 2445 7070 0    60   ~ 0
-RC16   LE_A\nRC17   LE_C\nRC18   LE_D\nRC19   RESET\nRC20   CLK\nRC21   DAT_DIR\nRC22   LED_POWER\nRC23   LED_CAPS\nRC24   INT\nRC25   WAIT\nRC26   LED_HAN\nRC27   SW1
+RC16   LE_A\nRC17   LE_C\nRC18   LE_D\nRC19   RESET\nRC20   CLK\nRC21   DAT_DIR\nRC22   LED_CODE\nRC23   LED_CAPS\nRC24   INT\nRC25   WAIT\nRC26   LED_HAN\nRC27   SW1
 $Comp
 L 74LS08 U7
@@
 RC26
 NoConn ~ 10450 1345
-Text Label 8685 2095 0    60   ~ 0
-M1
 NoConn ~ 9150 3345
 $Comp
