File: rpmpv16/rpmpv1.sch (KiCad schematic (older format))
At the start: 18 parts, among them J1 RPi_GPIO, J2 Conn_01x04, P1 CONN_02X25, U1 74HC244, U2 74HC244, U3 74LS07, U4 74HC244, U5 LVC4245, U6 7400

Commit message: update for new kicad but not perfect
Parts:
- removed U2: 74HC244, Housings_SOIC:SOIC-20W_7.5x12.8mm_Pitch1.27mm, symbol 74HC244
- removed U6: 7400, Housings_SOIC:SOIC-14_3.9x8.7mm_Pitch1.27mm, symbol 7400
- added U6: 74HC00, Package_SO:SOIC-14_3.9x8.7mm_P1.27mm, symbol 74xx:74HC00
- C1: symbol CP -> Device:CP
- C2: symbol C -> Device:C
- D1: symbol LED_RGB -> Device:LED_RGB
- J1: symbol RPi_GPIO -> rpi:RPi_GPIO
- J2: footprint Pin_Headers:Pin_Header_Angled_1x04_Pitch2.54mm -> Connector_PinHeader_2.54mm:PinHeader_1x04_P2.54mm_Horizontal; symbol Conn_01x04 -> Connector_Generic:Conn_01x04
- P1: symbol CONN_02X25 -> msx:CONN_02X25
- R1, R2, R3, R4, R5: symbol R -> Device:R
- U1, U4: symbol 74HC244 -> 74xx:74HC244
- U3: footprint Housings_SOIC:SOIC-14_3.9x8.7mm_Pitch1.27mm -> Package_SO:SOIC-14_3.9x8.7mm_P1.27mm; symbol 74LS05 -> 74xx:74LS07
- U5: symbol LVC4245 -> msx:LVC4245
- gave numbers to parts that had none: 1
Connections:
- net labels added: +3V3
- net labels removed: power_+3.3V
- wire segments 215 -> 242
- no-connect marks 11 -> 12

Commit message: new board with lichee pi nano
Parts:
- removed J1: RPi_GPIO, Socket_Strips:Socket_Strip_Angled_2x20_Pitch2.54mm, symbol rpi:RPi_GPIO
- removed U6: 74HC00, Package_SO:SOIC-14_3.9x8.7mm_P1.27mm, symbol 74xx:74HC00
- added R6, R7: R, Resistor_SMD:R_0805_2012Metric_Pad1.15x1.40mm_HandSolder, symbol Device:R
- added U6: licheepi_nano, MSX:licheepi_nano, symbol msx:licheepi_nano
- C1: footprint Capacitors_SMD:CP_Elec_4x4.5 -> Capacitor_THT:CP_Radial_Tantal_D5.0mm_P5.00mm
- C2: footprint Capacitors_SMD:C_0603_HandSoldering -> Capacitor_SMD:C_0805_2012Metric_Pad1.15x1.40mm_HandSolder
- R4, R5: footprint Resistors_SMD:R_0603_HandSoldering -> Resistor_SMD:R_0805_2012Metric_Pad1.15x1.40mm_HandSolder
Connections:
- net labels added: 3V3, INTR, RCLK, RINT, RIORQ, RMREQ, RRST, RWAIT, TVOUT
- net labels removed: +3V3, +5V, CWAIT, RC17, RC19, RC20, RC21, RC23, RC24, RC26, RC27
- wire segments 242 -> 223
- no-connect marks 12 -> 9

Commit message: more test pcb
Connections:
- net labels removed: 3V3
- wire segments 223 -> 224
Changed lines of the file:
@@
 	2250 6450 2600 6450
 Text Label 2350 6450 0    60   ~ 0
-3V3
+VCC
+Text Label 4200 5700 3    60   ~ 0
+GND
+Wire Wire Line
+	2050 3950 2050 4450
+Text Label 2050 4350 1    60   ~ 0
+VCC
 $EndSCHEMATC
