File: rpmpv18/rpmpv1.sch (KiCad schematic (older format))
At the start: 18 parts, among them J2 Conn_01x04, P1 CONN_02X25, U1 74HC244, U2 74HC244, U3 74LS07, U4 74HC244, U5 LVC4245

Commit message: sipeed m1 module
Connections:
- net labels added: BOOT, PCM_DATA, PCM_RCK, PCM_WS, RC17, RC19, RC20, RC21, RC23, RC24, SPI0_MISO, SPI0_MOSI, SPIO_CS, SPIO_SCLK, UARTRX, UARTTX, WIFI_EN, WIFI_RX, WIFI_TX
- net labels removed: TVOUT
- wire segments 205 -> 237
- no-connect marks 9 -> 40
Other:
- note added: "RC16 DAT_EN\nRC17 INT\nRC18 DAT_DIR\nRC19 WAIT\nRC20 \nRC21 MREQ"
- note added: "RC22 ADDR\nRC23 IORQ\nRC24 CLK\nRC25 RESET\n"
- note removed: "RC16 DAT_EN\nRC17 SLTSL\nRC18 SNDOUT\nRC19 IORQ\nRC20 RD\nRC21 M1"
- note removed: "RC22 ADDR\nRC23 INTR\nRC24 WAIT\nRC25 DAT_DIR\nRC26 MREQ\nRC27 WR"

Commit message: RPMP with sipeed m1w
Parts:
- added J1: Micro_SD_Card, MSX:Conn_uSDcard, symbol Connector:Micro_SD_Card
- added J3: Conn_01x04_Male, Connector_PinHeader_2.54mm:PinHeader_1x04_P2.54mm_Vertical, symbol Connector:Conn_01x04_Male
- added U7: PT8211, Package_SO:SOIC-8_3.9x4.9mm_P1.27mm, symbol MSX:PT8211
- added W1, W2: TEST, MSX:TestPoint_Pad_D1.0mm, symbol MSX:TEST
- J2: footprint Connector_PinHeader_2.54mm:PinHeader_1x04_P2.54mm_Horizontal -> Connector_PinHeader_2.54mm:PinHeader_1x04_P2.54mm_Vertical
- U6: renamed from U?; footprint (none) -> MSX:sipeed_m1
Connections:
- net labels added: SCL, SDN0, SND, SND0
- wire segments 237 -> 239
- no-connect marks 40 -> 39
Other:
- note added: "RPMP V1.9"
- note added: "RPMP V1.9 + Sipeed M1W"
- note removed: "RPMP V1.9 only with 74LVC4245 and some logics"

Commit message: updates for K210/F1C100S
Connections:
- net labels removed: SDN0
Changed lines of the file:
@@
 	3250 5350 3600 5350
 Text Label 3300 5350 0    60   ~ 0
-SDN0
+SND0
 Text Label 6000 5300 0    60   ~ 0
 SND0

Commit message: more test pcb
Parts:
- U7: symbol MSX:PT8211 -> rpmpv1-rescue:PT8211-MSX
- W1, W2: symbol MSX:TEST -> rpmpv1-rescue:TEST-MSX
Changed lines of the file:
@@
 NoConn ~ 3350 1500
 $Comp
-L MSX:PT8211 U7
+L rpmpv1-rescue:PT8211-MSX U7
 U 1 1 5E813C25
 P 5400 5400
@@
 NoConn ~ 5900 5400
 $Comp
-L MSX:TEST W1
+L rpmpv1-rescue:TEST-MSX W1
 U 1 1 5E8FD30E
 P 3050 5350
@@
 	5500 4300 5900 4300
 $Comp
-L MSX:TEST W2
+L rpmpv1-rescue:TEST-MSX W2
 U 1 1 5EBAEF55
 P 1250 5025
@@
 Text Label 2900 5650 0    60   ~ 0
 SND
+Text Label 4150 5900 0    60   ~ 0
+GND
 $EndSCHEMATC
