File: rpmpv2020.6/rpmpv1.kicad_pcb (KiCad board)
At the start: 2 copper layers, 99 x 64.4 mm, 19 parts, among them J1 RPi_GPIO, P1 CONN_02X25, U1 74HC244, U2 74HC244, U3 74LS07, U4 74HC244, U5 LVC4245

Commit message: updated for test
Parts:
- added U6: PT8211, Package_SO:SOIC-8_3.9x4.9mm_P1.27mm, F.Cu at (119.5, 87.1)
- added W1: TEST, MSX:TestPoint_Pad_D1.0mm, F.Cu at (112.4, 84.7)
- C1: value CP(10u) -> C(33n); footprint Capacitor_SMD:CP_Elec_4x4.5 -> Capacitor_SMD:C_0603_1608Metric
- C2: value C(33n) -> CP(10u); footprint Capacitor_SMD:C_0603_1608Metric -> Capacitor_SMD:CP_Elec_4x4.5; moved to F.Cu
- R4, R5: moved to F.Cu
- moved R4 11.3 mm to (112.4, 89.8), turned to 90 degrees
- moved R5 8.07 mm to (122.0, 93.7), turned to 180 degrees
- moved C1 5.62 mm to (117.0, 93.7)
- moved C2 3.51 mm to (119.5, 99.4), turned to 0 degrees
Connections:
- C1 pad 1: Net-(C1-Pad1) -> GND
- C1 pad 2: /SOUNDIN -> Net-(C1-Pad2)
- C2 pad 1: GND -> Net-(C1-Pad2)
- C2 pad 2: Net-(C1-Pad1) -> /SOUNDIN
- R4 pad 1: Net-(C1-Pad1) -> Net-(C1-Pad2)
- R4 pad 2: /RC18 -> /SND
- U4 pad 1: GND -> /DAT_EN
- U4 pad 11: /RESET -> /SLTSL
- U4 pad 12: /RC20 -> /RA15
- U4 pad 13: /SLTSL -> /MREQ
- U4 pad 14: /RC27 -> /RA14
- U4 pad 15: /MREQ -> /IORQ
- U4 pad 16: /RC21 -> /RA13
- U4 pad 17: /IORQ -> /RD
- U4 pad 3: /RC19 -> /RC20
- U4 pad 5: /RC26 -> /RC27
- U4 pad 7: /RC17 -> /RC26
- U4 pad 8: /RD -> /RESET
- U4 pad 9: Net-(U4-Pad9) -> /RC17
Routing:
- net /DAT_EN: track 73.5 -> 103.5 mm, vias 0 -> 1
- net /RC21: track 52.8 -> 28.6 mm, vias 1 -> 0
- net /RA13: track 38.6 -> 56.3 mm, vias 1 -> 3
- net /RD0: track 46.2 -> 63.7 mm, vias 2 -> 0
- net /A10: track 28.6 -> 44.1 mm
- net +3V3: track 132.0 -> 145.4 mm
- net Net-(C1-Pad2): track 0.00 -> 13.1 mm
- net /A7: track 20.6 -> 30.8 mm
- net /RD: track 14.3 -> 23.3 mm, vias 0 -> 2
- net /RESET: track 24.7 -> 16.0 mm
- net /ADDR: track 83.3 -> 91.1 mm, vias 1 -> 2
- net /SND: track 0.00 -> 7.67 mm
- net Net-(C1-Pad1): track 7.51 -> 0.00 mm, vias 1 -> 0
- net /RD5: track 41.6 -> 49.0 mm, vias 1 -> 0
- net /RD4: track 59.2 -> 66.5 mm, vias 3 -> 2
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Other:
- board text added: "2020.5.21"
- board text added: "2020.6"
- board text removed: "2020.5.20"
