File: rpmc_epm240/rpmc_epm240.kicad_pcb (KiCad board)
At the start: 2 copper layers, 90.3 x 52.3 mm, 9 parts, among them J1 Conn_02x20_Odd_Even, J2 Raspberry_Pi_2_3, U1 EPM240T100

Commit message: rpmc_epm240.kicad_pcb
Routing:
- net GND: track 272.5 -> 0.00 mm
- net +3V3: track 156.6 -> 0.00 mm, vias 2 -> 0
- net +5V: track 101.0 -> 0.00 mm
- net /A14: track 93.0 -> 0.00 mm
- net /BCK: track 87.1 -> 0.00 mm
- net /GCLK_OUT: track 78.9 -> 0.00 mm
- net /G0: track 75.3 -> 0.00 mm, vias 1 -> 0
- net /MREQ: track 62.2 -> 0.00 mm
- net /WAIT: track 58.6 -> 0.00 mm, vias 2 -> 0
- net /G2: track 53.4 -> 0.00 mm, vias 1 -> 0
- net /A15: track 52.8 -> 0.00 mm, vias 1 -> 0
- net /RD: track 52.5 -> 0.00 mm, vias 1 -> 0
- net /G3: track 50.5 -> 0.00 mm, vias 1 -> 0
- net /SOUNDIN: track 49.5 -> 0.00 mm
- net /G4: track 48.0 -> 0.00 mm, vias 1 -> 0
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
Commit message: pcb
Parts:
- moved R1 14.0 mm to (147.1, 75.7)
- moved R2 14.0 mm to (147.1, 77.5)
- moved R3 14.0 mm to (147.1, 79.2)
- moved R4 14.0 mm to (147.1, 81.0)
- moved JTAG1 14.0 mm to (151.5, 73.3)
Connections:
- JTAG1 pad 1: Net-(JTAG1-Pin_1) -> /TCK
- JTAG1 pad 3: Net-(JTAG1-Pin_3) -> /TDO
- JTAG1 pad 5: Net-(JTAG1-Pin_5) -> /TMS
- JTAG1 pad 9: Net-(JTAG1-Pin_9) -> /TDI
- R1 pad 2: Net-(JTAG1-Pin_1) -> /TCK
- R2 pad 2: Net-(JTAG1-Pin_3) -> /TDO
- R3 pad 2: Net-(JTAG1-Pin_5) -> /TMS
- R4 pad 2: Net-(JTAG1-Pin_9) -> /TDI
Routing:
- net GND: track 0.00 -> 275.6 mm, vias 0 -> 1
- net +3V3: track 0.00 -> 203.0 mm
- net +5V: track 0.00 -> 115.2 mm
- net /BCK: track 0.00 -> 84.2 mm
- net /GCLK_OUT: track 0.00 -> 76.0 mm, vias 0 -> 2
- net /MREQ: track 0.00 -> 69.2 mm, vias 0 -> 1
- net /WR: track 0.00 -> 68.9 mm
- net /WAIT: track 0.00 -> 65.9 mm, vias 0 -> 1
- net /G2: track 0.00 -> 64.7 mm, vias 0 -> 1
- net /SLTSL_1: track 0.00 -> 55.5 mm
- net /G3: track 0.00 -> 55.3 mm, vias 0 -> 1
- net /G4: track 0.00 -> 55.0 mm, vias 0 -> 1
- net /SOUNDIN: track 0.00 -> 49.5 mm
- net /GCLK: track 0.00 -> 48.3 mm, vias 0 -> 2
- net /RD: track 0.00 -> 48.1 mm, vias 0 -> 2
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
Commit message: libraries/footprint/FT2232H_EVB.kicad_mod libraries/footprint/SOIC-16_L10.8-W4.5-P1.27-LS6.8-BL.kicad_mod libraries/footprint/SOIC-20_L13.0-W7.6-P1.27-LS10.3-BL.kicad_mod libraries/msx_slot.kicad_sym rpmc_epm240/rpmc_epm240-backups/rpmc_epm240-2024-09-23_005415.zip rpmc_epm240/rpmc_epm240-backups/rpmc_epm240-2024-09-23_231002.zip rpmc_epm240/rpmc_epm240-backups/rpmc_epm240-2024-09-23_232423.zip rpmc_epm240/rpmc_epm240.kicad_pcb rpmc_epm240/rpmc_epm240.kicad_prl rpmc_ft2232h/fp-info-cache rpmc_ft2232h/fp-lib-table rpmc_ft2232h/rpmc_ft2232h-backups/rpmc_ft2232h-2024-09-24_003425.zip rpmc_ft2232h/rpmc_ft2232h-backups/rpmc_ft2232h-2024-09-24_010533.zip rpmc_ft2232h/rpmc_ft2232h-backups/rpmc_ft2232h-2024-09-24_011548.zip rpmc_ft2232h/rpmc_ft2232h.kicad_pcb rpmc_ft2232h/rpmc_ft2232h.kicad_prl rpmc_ft2232h/rpmc_ft2232h.kicad_pro rpmc_ft2232h/rpmc_ft2232h.kicad_sch rpmc_ft2232h/sym-lib-table rpmc_logics/sym-lib-table
Routing:
- added copper zone on B.Cu, net GND
- added copper zone on F.Cu, net GND
Other:
- board text added: "2024-09-23"
- board text added: "RPMC_EPM240"
Changed lines of the file:
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@@
 		(tags "resistor handsolder")
 		(property "Reference" "R2"
-			(at 0 -1.05 0)
+			(at -2.0675 0.04 0)
 			(layer "F.SilkS")
 			(effects
@@
 		(tags "resistor handsolder")
 		(property "Reference" "R4"
-			(at 0 -1.05 0)
+			(at -2.0675 0.54 0)
 			(layer "F.SilkS")
 			(effects
@@
 		(tags "resistor handsolder")
 		(property "Reference" "R3"
-			(at 0 -1.05 0)
+			(at -2.0675 0.29 0)
 			(layer "F.SilkS")
 			(effects
@@
 		(tags "resistor handsolder")
 		(property "Reference" "R1"
-			(at 0 -1.05 0)
+			(at -2.0675 -0.21 0)
 			(layer "F.SilkS")
 			(effects
@@
 		(layer "Edge.Cuts")
 	)
+	(gr_text "2024-09-23"
+		(at 68 95.5 0)
+		(layer "F.SilkS")
+		(effects
+			(font
+				(size 2 2)
+				(thickness 0.1)
+			)
+			(justify left bottom)
+		)
+	)
+	(gr_text "RPMC_EPM240"
+		(at 68 92 0)
+		(layer "F.SilkS")
+		(effects
+			(font
+				(size 1 1)
+				(thickness 0.1)
+			)
+			(justify left bottom)
+		)
+	)
 	(segment
 		(start 123.5 63.325)
@@
 	(segment
 		(start 115.38 91.46)
-		(end 115.38 90.3083)
+		(end 115.38 88.2734)
 		(width 0.2)
 		(layer "B.Cu")
@@
 	)
 	(segment
-		(start 115.38 90.3083)
-		(end 115.38 88.2734)
-		(width 0.2)
-		(layer "B.Cu")
-		(net 3)
-	)
-	(segment
 		(start 119.937 73.7787)
 		(end 119.937 63.4842)
@@
 	)
 	(segment
-		(start 128.08 90.3083)
+		(start 128.08 91.46)
 		(end 128.08 89.7404)
 		(width 0.2)
@@
 	)
 	(segment
-		(start 128.08 91.46)
-		(end 128.08 90.3083)
-		(width 0.2)
-		(layer "B.Cu")
-		(net 15)
-	)
-	(segment
 		(start 118.5218 61.8106)
 		(end 119 62.2888)
@@
 	(segment
 		(start 105.22 91.46)
-		(end 105.22 90.3083)
+		(end 105.22 76.9524)
 		(width 0.2)
 		(layer "B.Cu")
@@
 	)
 	(segment
-		(start 105.22 90.3083)
-		(end 105.22 76.9524)
-		(width 0.2)
-		(layer "B.Cu")
-		(net 36)
-	)
-	(segment
 		(start 105.22 76.9524)
 		(end 107.5636 74.6088)
@@
 	)
 	(segment
-		(start 107.76 90.3083)
-		(end 107.76 81.0899)
-		(width 0.2)
-		(layer "B.Cu")
-		(net 37)
-	)
-	(segment
 		(start 107.76 91.46)
-		(end 107.76 90.3083)
+		(end 107.76 81.0899)
 		(width 0.2)
 		(layer "B.Cu")
@@
 	(segment
 		(start 120.38 51.54)
-		(end 120.38 52.6917)
+		(end 120.38 58.0137)
 		(width 0.2)
 		(layer "B.Cu")
@@
 	)
 	(segment
-		(start 120.38 58.0137)
-		(end 120.38 52.6917)
-		(width 0.2)
-		(layer "B.Cu")
-		(net 62)
-	)
-	(segment
 		(start 123.6744 65.7949)
 		(end 123.6744 63.7195)
@@
 	)
 	(segment
-		(start 151.46 75.88)
-		(end 150.3083 75.88)
+		(start 148.5144 75.88)
+		(end 151.46 75.88)
 		(width 0.2)
 		(layer "F.Cu")
@@
 	)
 	(segment
-		(start 148.5144 75.88)
-		(end 150.3083 75.88)
-		(width 0.2)
-		(layer "F.Cu")
-		(net 96)
-	)
-	(segment
 		(start 148.1421 77.977)
 		(end 147.0922 77.977)
@@
 		(net 99)
 	)
+	(zone
+		(net 6)
+		(net_name "GND")
+		(layer "F.Cu")
+		(hatch edge 0.5)
+		(connect_pads
+			(clearance 0.5)
+		)
+		(min_thickness 0.25)
+		(filled_areas_thickness no)
+		(fill yes
+			(thermal_gap 0.5)
+			(thermal_bridge_width 0.5)
+		)
+		(polygon
+			(pts
+				(xy 64.5 43.5) (xy 64 99) (xy 159 99) (xy 158.5 44)
+			)
+		)
+	)
+	(zone
+		(net 6)
+		(net_name "GND")
+		(layer "B.Cu")
+		(hatch edge 0.5)
+		(priority 1)
+		(connect_pads
+			(clearance 0.5)
+		)
+		(min_thickness 0.25)
+		(filled_areas_thickness no)
+		(fill yes
+			(thermal_gap 0.5)
+			(thermal_bridge_width 0.5)
+		)
+		(polygon
+			(pts
+				(xy 64 43) (xy 64 100) (xy 159 100) (xy 159 42.5)
+			)
+		)
+	)
 )

Commit message: epm240
Connections:
- J2 pad 13: unconnected-(J2-GPIO27-Pad13) -> /G27
- J2 pad 15: unconnected-(J2-GPIO22-Pad15) -> /G22
- J2 pad 16: unconnected-(J2-GPIO23-Pad16) -> /G23
- J2 pad 18: unconnected-(J2-GPIO24-Pad18) -> /G24
- J2 pad 22: unconnected-(J2-GPIO25-Pad22) -> /G25
- J2 pad 37: unconnected-(J2-GPIO26-Pad37) -> /G26
- U1 pad 33: unconnected-(U1-IO1_33-Pad33) -> /G22
- U1 pad 34: unconnected-(U1-IO1_34-Pad34) -> /G23
- U1 pad 35: unconnected-(U1-IO1_35-Pad35) -> /G24
- U1 pad 36: unconnected-(U1-IO1_36-Pad36) -> /G25
- U1 pad 37: unconnected-(U1-IO1_37-Pad37) -> /G26
- U1 pad 38: unconnected-(U1-IO1_38-Pad38) -> /G27
- U2 pad 12: (no net) -> /LRC
Routing:
- net /LRC: track 0.00 -> 47.5 mm
- net /G26: track 0.00 -> 47.4 mm, vias 0 -> 2
- net /A15: track 45.1 -> 82.2 mm, vias 2 -> 1
- net /WR: track 68.9 -> 33.2 mm, vias 0 -> 1
- net /A14: track 45.1 -> 72.0 mm, vias 2 -> 1
- net /G22: track 0.00 -> 26.7 mm, vias 0 -> 1
- net /G25: track 0.00 -> 25.1 mm, vias 0 -> 1
- net /G24: track 0.00 -> 24.6 mm, vias 0 -> 1
- net /G27: track 0.00 -> 24.4 mm, vias 0 -> 1
- net /G23: track 0.00 -> 23.6 mm, vias 0 -> 1
- net /MREQ: track 69.2 -> 92.2 mm
- net /A2: track 43.9 -> 28.6 mm
- net /G10: track 35.8 -> 50.4 mm
- net +5V: track 115.2 -> 101.0 mm
- net /A10: track 30.1 -> 43.4 mm
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Other:
- board text removed: "2024-09-23"
- board text removed: "RPMC_EPM240"
