File: epm240_msxcart/epm240_msxcart.kicad_pcb (KiCad board)
At the start: 2 copper layers, 103 x 65 mm, 10 parts, among them J1 Conn_01x21_Pin, P1 CONN_02X25, U1 EPM240T100, U2 AP1117-33, X1 TXC-7C

Commit message: epm240_msxcart/epm240_msxcart.kicad_pcb epm240_msxcart/epm240_msxcart.kicad_prl epm240_msxcart/epm240_msxcart.kicad_sch epm240_msxcart/fp-info-cache epm240_msxcart/freerouting.dsn epm240_msxcart/freerouting.ses universal_msxcart/.gitignore universal_msxcart/fp-info-cache universal_msxcart/universal_msxcart.kicad_pcb universal_msxcart/universal_msxcart.kicad_prl universal_msxcart/universal_msxcart.kicad_sch
Parts:
- removed U2: AP1117-33, Package_TO_SOT_SMD:SOT-223-3_TabPin2
Routing:
- net GND: track 0.00 -> 223.5 mm
- net +3V3: track 0.00 -> 177.7 mm
- net /TDI: track 0.00 -> 83.1 mm
- net /A0: track 0.00 -> 71.9 mm
- net /+5V: track 0.00 -> 63.6 mm
- net /WAIT: track 0.00 -> 59.1 mm, vias 0 -> 1
- net /INT: track 0.00 -> 58.2 mm, vias 0 -> 2
- net /SOUNDIN: track 0.00 -> 57.2 mm
- net /IORQ: track 0.00 -> 56.5 mm, vias 0 -> 1
- net /BUSDIR: track 0.00 -> 55.1 mm, vias 0 -> 2
- net /WR: track 0.00 -> 54.0 mm, vias 0 -> 1
- net /M1: track 0.00 -> 53.7 mm, vias 0 -> 1
- net /TMS: track 0.00 -> 51.8 mm, vias 0 -> 1
- net /RESET: track 0.00 -> 51.3 mm, vias 0 -> 1
- net /TDO: track 0.00 -> 51.0 mm, vias 0 -> 1
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